File: boards/daq-node/CAN_Transceiver_sch.kicad_sch (KiCad schematic)
At the start: 10 parts, among them J8 917780-1, U2 TJA1051T-3, U4 TPD2EUSB30, U5 ACT45B-101-2P-TL003

Commit message: Add auxiliary boards to harness; fix daq + hud ERC errors
Harness / diagram:
- Support repeated boards in the car diagram by importing one generated
  YAML under multiple include aliases; the renderer now namespaces each
  component's layout zone by its alias so instances get their own column
  (harness/wirelab/parser.py).
- Add wheel-hall (x4), fuel-sensor, and ecvt-hall aux boards as
  hand-written placeholder generated/*.yaml, instanced and wired in
  car.yaml (front wheels -> HUD J5, rear -> daq J7, eCVT halls -> ecvt J3,
  fuel -> daq J4). Documented the pattern in harness/README.md.
- extract_connectors.py now also identifies off-board connectors by
  footprint family, so a connector whose Value is left generic
  (e.g. Conn_01x04) but whose footprint is a 917xxx/Molex part is no
  longer dropped. This recovered HUD J5 (wheel power).

Board ERC fixes:
- daq-node: resolve ERC errors (dangling GPIO labels, undriven power
  pin, power-flag conflicts).
- hud-node: finish the +3.3V -> +3V3 power-symbol rename across all
  sheets (MCU sheet was missed), which had split the 3.3V net and left
  an undriven power pin on the Can sheet.

Co-Authored-By: Claude Opus 4.8 <noreply@anthropic.com>
Changed lines of the file:
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@@
-	)
-	(junction
-		(at 59.69 107.95)
-		(diameter 0)
-		(color 0 0 0 0)
 	)
 	(junction
@@
 	(wire
 		(pts
-			(xy 55.88 107.95) (xy 59.69 107.95)
+			(xy 55.88 107.95) (xy 67.31 107.95)
 		)
 		(stroke
@@
 	(wire
 		(pts
-			(xy 59.69 104.14) (xy 59.69 107.95)
-		)
-		(stroke
-			(width 0)
-			(type default)
-		)
-	)
-	(wire
-		(pts
 			(xy 146.05 118.11) (xy 146.05 116.84)
 		)
@@
 		(pts
 			(xy 100.33 73.66) (xy 100.33 74.93)
-		)
-		(stroke
-			(width 0)
-			(type default)
-		)
-	)
-	(wire
-		(pts
-			(xy 59.69 107.95) (xy 67.31 107.95)
 		)
 		(stroke
@@
 					(unit 1)
 				)
-			)
-		)
-	)
-	(symbol
-		(lib_id "power:PWR_FLAG")
-		(at 59.69 104.14 0)
-		(unit 1)
-		(exclude_from_sim no)
-		(in_bom yes)
-		(on_board yes)
-		(dnp no)
-		(property "Reference" "#FLG05"
-			(at 59.69 102.235 0)
-			(effects
-				(font
-					(size 1.27 1.27)
-				)
-				(hide yes)
-			)
-		)
-		(property "Value" "PWR_FLAG"
-			(at 59.69 99.822 0)
-			(effects
-				(font
-					(size 1.27 1.27)
-				)
-			)
-		)
-		(property "Footprint" ""
-			(at 59.69 104.14 0)
-			(effects
-				(font
-					(size 1.27 1.27)
-				)
-				(hide yes)
-			)
-		)
-		(property "Datasheet" "~"
-			(at 59.69 104.14 0)
-			(effects
-				(font
-					(size 1.27 1.27)
-				)
-				(hide yes)
-			)
-		)
-		(property "Description" "Special symbol for telling ERC where power comes from"
-			(at 59.69 104.14 0)
-			(effects
-				(font
-					(size 1.27 1.27)
-				)
-				(hide yes)
-			)
-		)
-		(pin "1"
-		)
-		(instances
-			(project "daq_board"
-				(path "/fbbff63c-816e-460c-8c40-59811440d581/de124adb-cf0a-42c7-9406-ce6718e339ee"
-					(reference "#FLG05")
-					(unit 1)
-				)
