File: boards/daq-node/power_circuitry.kicad_sch (KiCad schematic)
At the start: 10 parts, among them J5 15311026, Q1 Q_PMOS_DGS, U3 TSR_1-2450

Commit message: Add auxiliary boards to harness; fix daq + hud ERC errors
Harness / diagram:
- Support repeated boards in the car diagram by importing one generated
  YAML under multiple include aliases; the renderer now namespaces each
  component's layout zone by its alias so instances get their own column
  (harness/wirelab/parser.py).
- Add wheel-hall (x4), fuel-sensor, and ecvt-hall aux boards as
  hand-written placeholder generated/*.yaml, instanced and wired in
  car.yaml (front wheels -> HUD J5, rear -> daq J7, eCVT halls -> ecvt J3,
  fuel -> daq J4). Documented the pattern in harness/README.md.
- extract_connectors.py now also identifies off-board connectors by
  footprint family, so a connector whose Value is left generic
  (e.g. Conn_01x04) but whose footprint is a 917xxx/Molex part is no
  longer dropped. This recovered HUD J5 (wheel power).

Board ERC fixes:
- daq-node: resolve ERC errors (dangling GPIO labels, undriven power
  pin, power-flag conflicts).
- hud-node: finish the +3.3V -> +3V3 power-symbol rename across all
  sheets (MCU sheet was missed), which had split the 3.3V net and left
  an undriven power pin on the Can sheet.

Co-Authored-By: Claude Opus 4.8 <noreply@anthropic.com>
Changed lines of the file:
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@@
+	)
+	(junction
+		(at 113.03 68.58)
+		(diameter 0)
+		(color 0 0 0 0)
 	)
 	(junction
@@
 	)
 	(junction
-		(at 156.21 68.58)
-		(diameter 0)
-		(color 0 0 0 0)
-	)
-	(junction
 		(at 52.07 71.12)
 		(diameter 0)
@@
 	(wire
 		(pts
-			(xy 109.22 68.58) (xy 114.3 68.58)
+			(xy 109.22 68.58) (xy 113.03 68.58)
 		)
 		(stroke
@@
 	(wire
 		(pts
-			(xy 156.21 62.23) (xy 156.21 68.58)
-		)
-		(stroke
-			(width 0)
-			(type default)
-		)
-	)
-	(wire
-		(pts
 			(xy 77.47 83.82) (xy 77.47 86.36)
 		)
@@
 		(pts
 			(xy 82.55 68.58) (xy 87.63 68.58)
+		)
+		(stroke
+			(width 0)
+			(type default)
+		)
+	)
+	(wire
+		(pts
+			(xy 113.03 68.58) (xy 114.3 68.58)
 		)
 		(stroke
@@
 	)
 	(symbol
-		(lib_id "power:PWR_FLAG")
-		(at 156.21 62.23 0)
-		(unit 1)
-		(exclude_from_sim no)
-		(in_bom yes)
-		(on_board yes)
-		(dnp no)
-		(property "Reference" "#FLG03"
-			(at 156.21 60.325 0)
-			(effects
-				(font
-					(size 1.27 1.27)
-				)
-				(hide yes)
-			)
-		)
-		(property "Value" "PWR_FLAG"
-			(at 156.464 58.42 0)
-			(effects
-				(font
-					(size 1.27 1.27)
-				)
-			)
-		)
-		(property "Footprint" ""
-			(at 156.21 62.23 0)
-			(effects
-				(font
-					(size 1.27 1.27)
-				)
-				(hide yes)
-			)
-		)
-		(property "Datasheet" "~"
-			(at 156.21 62.23 0)
-			(effects
-				(font
-					(size 1.27 1.27)
-				)
-				(hide yes)
-			)
-		)
-		(property "Description" "Special symbol for telling ERC where power comes from"
-			(at 156.21 62.23 0)
-			(effects
-				(font
-					(size 1.27 1.27)
-				)
-				(hide yes)
-			)
-		)
-		(pin "1"
-		)
-		(instances
-			(project "daq_board"
-				(path "/fbbff63c-816e-460c-8c40-59811440d581/a07dad94-c479-404c-ab65-d7eb79233e52"
-					(reference "#FLG03")
-					(unit 1)
-				)
-			)
-		)
-	)
-	(symbol
 		(lib_id "power:GND")
 		(at 140.97 76.2 0)
@@
 					(unit 1)
 				)
+			)
+		)
+	)
+	(symbol
+		(lib_id "power:PWR_FLAG")
+		(at 113.03 68.58 0)
+		(unit 1)
+		(exclude_from_sim no)
+		(in_bom yes)
+		(on_board yes)
+		(dnp no)
+		(property "Reference" "#FLG07"
+			(at 113.03 66.675 0)
+			(effects
+				(font
+					(size 1.27 1.27)
+				)
+				(hide yes)
+			)
+		)
+		(property "Value" "PWR_FLAG"
+			(at 113.284 64.77 0)
+			(effects
+				(font
+					(size 1.27 1.27)
+				)
+			)
+		)
+		(property "Footprint" ""
+			(at 113.03 68.58 0)
+			(effects
+				(font
+					(size 1.27 1.27)
+				)
+				(hide yes)
+			)
+		)
+		(property "Datasheet" "~"
+			(at 113.03 68.58 0)
+			(effects
+				(font
+					(size 1.27 1.27)
+				)
+				(hide yes)
+			)
+		)
+		(property "Description" "Special symbol for telling ERC where power comes from"
+			(at 113.03 68.58 0)
+			(effects
+				(font
+					(size 1.27 1.27)
+				)
+				(hide yes)
+			)
+		)
+		(pin "1"
+		)
+		(instances
+			(project "daq_board"
+				(path "/fbbff63c-816e-460c-8c40-59811440d581/a07dad94-c479-404c-ab65-d7eb79233e52"
+					(reference "#FLG07")
+					(unit 1)
+				)
