File: boards/hud-node/Can.kicad_sch (KiCad schematic)
At the start: 10 parts, among them U2 TJA1051T-3, U3 ACT45B-101-2P-TL003, U5 TPD2EUSB30

Commit message: Add auxiliary boards to harness; fix daq + hud ERC errors
Harness / diagram:
- Support repeated boards in the car diagram by importing one generated
  YAML under multiple include aliases; the renderer now namespaces each
  component's layout zone by its alias so instances get their own column
  (harness/wirelab/parser.py).
- Add wheel-hall (x4), fuel-sensor, and ecvt-hall aux boards as
  hand-written placeholder generated/*.yaml, instanced and wired in
  car.yaml (front wheels -> HUD J5, rear -> daq J7, eCVT halls -> ecvt J3,
  fuel -> daq J4). Documented the pattern in harness/README.md.
- extract_connectors.py now also identifies off-board connectors by
  footprint family, so a connector whose Value is left generic
  (e.g. Conn_01x04) but whose footprint is a 917xxx/Molex part is no
  longer dropped. This recovered HUD J5 (wheel power).

Board ERC fixes:
- daq-node: resolve ERC errors (dangling GPIO labels, undriven power
  pin, power-flag conflicts).
- hud-node: finish the +3.3V -> +3V3 power-symbol rename across all
  sheets (MCU sheet was missed), which had split the 3.3V net and left
  an undriven power pin on the Can sheet.

Co-Authored-By: Claude Opus 4.8 <noreply@anthropic.com>
Connections:
- net +3.3V renamed +3V3
Changed lines of the file:
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@@
 			)
 		)
-		(property "Value" "+3.3V"
-			(at 71.12 88.9 0)
+		(property "Value" "+3V3"
+			(at 73.66 92.7099 0)
 			(effects
 				(font
 					(size 1.27 1.27)
 				)
+				(justify left)
 			)
 		)
