File: boards/ecvt-controller/ecvt-controller/CAN.kicad_sch (KiCad schematic)
At the start: 12 parts, among them SW1 SW_SPST, SW2 SW_SPST, U1 TJA1051T-3

Commit message: CAN
Parts:
- added U5: ACT45B-101-2P-TL003, baja_footprint_library:ACT45B-101-2P-TL003, symbol baja_symbol_library:ACT45B-101-2P-TL003
- added U6: PESD2CAN,215, Package_TO_SOT_SMD:SOT-23, symbol baja_symbol_library:ESD3V3AP-TP
- SW1, SW2: footprint (none) -> Button_Switch_THT:SW_DIP_SPSTx01_Slide_9.78x4.72mm_W7.62mm_P2.54mm
Connections:
- net CANH: now also U5.4 (OUT1)
- net CANL: now also U5.3 (OUT2)
- net GND: now also U6.3
- net at U1.6 (CANL): now also U5.2 (IN2), U6.2
- net at U1.7 (CANH): now also U5.1 (IN1), U6.1
Other:
- moved on the sheet: C7, C8, C9, R2, R3, SW1, SW2

Commit message: CAN actually done
Parts:
- added C10, C11: 22pF, symbol Device:C
- added R4: 10k, symbol Device:R
- added U3: MCP2515-xSO, Package_SO:SOIC-18W_7.5x11.6mm_P1.27mm, symbol Interface_CAN_LIN:MCP2515-xSO
- added Y1: Crystal, Crystal:Crystal_SMD_5032-2Pin_5.0x3.2mm_HandSoldering, symbol Device:Crystal
Connections:
- net +3.3V: now also R4.1, U3.18 (VDD)
- net GND: now also C10.1, C11.1, U3.9 (VSS)
- net RX: no longer names the net of U1.4 (RXD)
- net RX: now also U3.2 (RXCAN)
- net TX: no longer names the net of U1.1 (TXD)
- net TX: now also U3.1 (TXCAN)
- new net: R4.2, U3.17 (~{RESET})
- new net: C10.2, U3.7 (OSC2), Y1.1
- new net: C11.2, U3.8 (OSC1), Y1.2
- new net CS: U3.16 (~{CS})
- new net INT: U3.12 (~{INT})
- new net SCK: U3.13 (SCK)
- new net SI: U3.14 (SI)
- new net SO: U3.15 (SO)
Other:
- note added: "order 30-33pF as well just in case for the crystal caps"
- moved on the sheet: C3, C4, C5, C6, C7, C8, C9, R2, R3, SW1, SW2, U1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

Commit message: almost done schmatic
Other:
- moved on the sheet: C3, C4
Changed lines of the file:
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@@
 	)
 	(junction
-		(at 100.33 120.65)
+		(at 107.95 120.65)
 		(diameter 0)
 		(color 0 0 0 0)
@@
 	)
 	(junction
-		(at 111.76 120.65)
+		(at 119.38 120.65)
 		(diameter 0)
 		(color 0 0 0 0)
@@
 	(wire
 		(pts
-			(xy 115.57 100.33) (xy 137.16 100.33)
+			(xy 123.19 100.33) (xy 137.16 100.33)
 		)
 		(stroke
@@
 	(wire
 		(pts
-			(xy 100.33 120.65) (xy 97.79 120.65)
+			(xy 107.95 120.65) (xy 105.41 120.65)
 		)
 		(stroke
@@
 	(wire
 		(pts
-			(xy 115.57 120.65) (xy 111.76 120.65)
+			(xy 123.19 120.65) (xy 119.38 120.65)
 		)
 		(stroke
@@
 	(wire
 		(pts
-			(xy 115.57 120.65) (xy 115.57 100.33)
+			(xy 123.19 120.65) (xy 123.19 100.33)
 		)
 		(stroke
@@
 	(wire
 		(pts
-			(xy 97.79 107.95) (xy 97.79 120.65)
+			(xy 105.41 107.95) (xy 105.41 120.65)
 		)
 		(stroke
@@
 	(wire
 		(pts
-			(xy 111.76 120.65) (xy 100.33 120.65)
+			(xy 119.38 120.65) (xy 107.95 120.65)
 		)
 		(stroke
@@
 	(symbol
 		(lib_id "power:+3.3V")
-		(at 97.79 107.95 0)
+		(at 105.41 107.95 0)
 		(unit 1)
 		(body_style 1)
@@
 		(fields_autoplaced yes)
 		(property "Reference" "#PWR014"
-			(at 97.79 111.76 0)
+			(at 105.41 111.76 0)
 			(hide yes)
 			(show_name no)
@@
 		)
 		(property "Value" "+3.3V"
-			(at 97.79 102.87 0)
+			(at 105.41 102.87 0)
 			(show_name no)
 			(do_not_autoplace no)
@@
 		)
 		(property "Footprint" ""
-			(at 97.79 107.95 0)
+			(at 105.41 107.95 0)
 			(hide yes)
 			(show_name no)
@@
 		)
 		(property "Datasheet" ""
-			(at 97.79 107.95 0)
+			(at 105.41 107.95 0)
 			(hide yes)
 			(show_name no)
@@
 		)
 		(property "Description" "Power symbol creates a global label with name \"+3.3V\""
-			(at 97.79 107.95 0)
+			(at 105.41 107.95 0)
 			(hide yes)
 			(show_name no)
@@
 	(symbol
 		(lib_id "power:GND")
-		(at 100.33 128.27 0)
+		(at 107.95 128.27 0)
 		(unit 1)
 		(body_style 1)
@@
 		(fields_autoplaced yes)
 		(property "Reference" "#PWR017"
-			(at 100.33 134.62 0)
+			(at 107.95 134.62 0)
 			(hide yes)
 			(show_name no)
@@
 		)
 		(property "Value" "GND"
-			(at 100.33 133.35 0)
+			(at 107.95 133.35 0)
 			(show_name no)
 			(do_not_autoplace no)
@@
 		)
 		(property "Footprint" ""
-			(at 100.33 128.27 0)
+			(at 107.95 128.27 0)
 			(hide yes)
 			(show_name no)
@@
 		)
 		(property "Datasheet" ""
-			(at 100.33 128.27 0)
+			(at 107.95 128.27 0)
 			(hide yes)
 			(show_name no)
@@
 		)
 		(property "Description" "Power symbol creates a global label with name \"GND\" , ground"
-			(at 100.33 128.27 0)
+			(at 107.95 128.27 0)
 			(hide yes)
 			(show_name no)
@@
 	(symbol
 		(lib_id "Device:C")
-		(at 111.76 124.46 0)
+		(at 119.38 124.46 0)
 		(unit 1)
 		(body_style 1)
@@
 		(fields_autoplaced yes)
 		(property "Reference" "C4"
-			(at 115.57 123.1899 0)
+			(at 123.19 123.1899 0)
 			(show_name no)
 			(do_not_autoplace no)
@@
 		)
 		(property "Value" "C"
-			(at 115.57 125.7299 0)
+			(at 123.19 125.7299 0)
 			(show_name no)
 			(do_not_autoplace no)
@@
 		)
 		(property "Footprint" ""
-			(at 112.7252 128.27 0)
+			(at 120.3452 128.27 0)
 			(hide yes)
 			(show_name no)
@@
 		)
 		(property "Datasheet" ""
-			(at 111.76 124.46 0)
+			(at 119.38 124.46 0)
 			(hide yes)
 			(show_name no)
@@
 		)
 		(property "Description" "Unpolarized capacitor"
-			(at 111.76 124.46 0)
+			(at 119.38 124.46 0)
 			(hide yes)
 			(show_name no)
@@
 	(symbol
 		(lib_id "power:GND")
-		(at 111.76 128.27 0)
+		(at 119.38 128.27 0)
 		(unit 1)
 		(body_style 1)
@@
 		(fields_autoplaced yes)
 		(property "Reference" "#PWR018"
-			(at 111.76 134.62 0)
+			(at 119.38 134.62 0)
 			(hide yes)
 			(show_name no)
@@
 		)
 		(property "Value" "GND"
-			(at 111.76 133.35 0)
+			(at 119.38 133.35 0)
 			(show_name no)
 			(do_not_autoplace no)
@@
 		)
 		(property "Footprint" ""
-			(at 111.76 128.27 0)
+			(at 119.38 128.27 0)
 			(hide yes)
 			(show_name no)
@@
 		)
 		(property "Datasheet" ""
-			(at 111.76 128.27 0)
+			(at 119.38 128.27 0)
 			(hide yes)
 			(show_name no)
@@
 		)
 		(property "Description" "Power symbol creates a global label with name \"GND\" , ground"
-			(at 111.76 128.27 0)
+			(at 119.38 128.27 0)
 			(hide yes)
 			(show_name no)
@@
 	(symbol
 		(lib_id "Device:C")
-		(at 100.33 124.46 0)
+		(at 107.95 124.46 0)
 		(unit 1)
 		(body_style 1)
@@
 		(fields_autoplaced yes)
 		(property "Reference" "C3"
-			(at 104.14 123.1899 0)
+			(at 111.76 123.1899 0)
 			(show_name no)
 			(do_not_autoplace no)
@@
 		)
 		(property "Value" "C"
-			(at 104.14 125.7299 0)
+			(at 111.76 125.7299 0)
 			(show_name no)
 			(do_not_autoplace no)
@@
 		)
 		(property "Footprint" ""
-			(at 101.2952 128.27 0)
+			(at 108.9152 128.27 0)
 			(hide yes)
 			(show_name no)
@@
 		)
 		(property "Datasheet" ""
-			(at 100.33 124.46 0)
+			(at 107.95 124.46 0)
 			(hide yes)
 			(show_name no)
@@
 		)
 		(property "Description" "Unpolarized capacitor"
-			(at 100.33 124.46 0)
-			(hide yes)
-			(show_name no)
+			(at 107.95 124.46 0)
+			(hide yes)
+			(show_name no)

Commit message: cap sizing
Parts:
- C3, C5: value C -> 4.7 µF
- C4, C6, C7: value C -> 0.1 µF
- C8, C9: value C -> 220 pF
- R2, R3: value R -> 60
Connections:
- net +3.3V: no longer R4.1
Changed lines of the file:
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@@
 	)
 	(junction
-		(at 86.36 113.03)
-		(diameter 0)
-		(color 0 0 0 0)
-	)
-	(junction
 		(at 243.84 72.39)
 		(diameter 0)
@@
 	(wire
 		(pts
-			(xy 86.36 107.95) (xy 86.36 113.03)
-		)
-		(stroke
-			(width 0)
-			(type default)
-		)
-	)
-	(wire
-		(pts
 			(xy 123.19 120.65) (xy 123.19 100.33)
 		)
@@
 	(wire
 		(pts
-			(xy 86.36 113.03) (xy 86.36 114.3)
+			(xy 86.36 107.95) (xy 86.36 114.3)
 		)
 		(stroke
@@
 			)
 		)
-		(property "Value" "C"
+		(property "Value" "0.1 µF"
 			(at 162.56 76.1999 0)
 			(show_name no)
@@
 			)
 		)
-		(property "Value" "C"
+		(property "Value" "220 pF"
 			(at 273.05 124.4599 0)
 			(show_name no)
@@
 			)
 		)
-		(property "Value" "C"
+		(property "Value" "0.1 µF"
 			(at 123.19 125.7299 0)
 			(show_name no)
@@
 			)
 		)
-		(property "Value" "C"
+		(property "Value" "0.1 µF"
 			(at 260.35 101.5999 0)
 			(show_name no)
@@
 			)
 		)
-		(property "Value" "R"
+		(property "Value" "60"
 			(at 246.38 90.1699 0)
 			(show_name no)
@@
 			)
 		)
-		(property "Value" "C"
+		(property "Value" "4.7 µF"
 			(at 111.76 125.7299 0)
 			(show_name no)
@@
 			)
 		)
-		(property "Value" "R"
+		(property "Value" "60"
 			(at 246.38 101.5999 0)
 			(show_name no)
@@
 			)
 		)
-		(property "Value" "C"
+		(property "Value" "4.7 µF"
 			(at 142.24 76.1999 0)
 			(show_name no)
@@
 			)
 		)
-		(property "Value" "C"
+		(property "Value" "220 pF"
 			(at 271.78 77.4699 0)
 			(show_name no)

Commit message: components done. RAHHHHH
Parts:
- removed C3, C5: 4.7 µF, symbol Device:C
- removed C4, C6, C7: 0.1 µF, symbol Device:C
- removed C8, C9: 220 pF, symbol Device:C
- removed R2, R3: 60, symbol Device:R
- added C15, C17: 4.7µF, Capacitor_SMD:C_0603_1608Metric_Pad1.08x0.95mm_HandSolder, symbol Device:C
- added C16, C18, C21: 0.1 µF, Capacitor_SMD:C_0603_1608Metric_Pad1.08x0.95mm_HandSolder, symbol Device:C
- added C19, C20: 220 pF, Capacitor_SMD:C_0603_1608Metric_Pad1.08x0.95mm_HandSolder, symbol Device:C
- added R5, R6: 60, Resistor_SMD:R_1206_3216Metric_Pad1.30x1.75mm_HandSolder, symbol Device:R
- C10, C11: footprint (none) -> Capacitor_SMD:C_0805_2012Metric_Pad1.18x1.45mm_HandSolder
Connections:
- net +3.3V: now also C15.1, C16.1
- net +5V: now also C17.1, C18.1
- net CANH: now also C20.1
- net CANL: now also C19.1
- net GND: now also C15.2, C16.2, C17.2, C18.2, C19.2, C20.2, C21.1
- net at SW2.1 (A): now also R6.1
- net at SW1.2 (B): now also R5.2
- new net: C21.2, R5.1, R6.2

Commit message: initial placement
Parts:
- R4: footprint (none) -> Resistor_SMD:R_0603_1608Metric_Pad0.98x0.95mm_HandSolder
Connections:
- net S is gone; now on net GND: U1.8 (S)
- net +3.3V: now also R4.1
Other:
- moved on the sheet: R4
Changed lines of the file:
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@@
-	(wire
-		(pts
-			(xy 86.36 120.65) (xy 86.36 121.92)
-		)
-		(stroke
-			(width 0)
-			(type default)
-		)
-	)
 	(wire
 		(pts
@@
 			)
 			(justify left)
-		)
-	)
-	(hierarchical_label "S"
-		(shape input)
-		(at 130.81 102.87 180)
-		(effects
-			(font
-				(size 1.27 1.27)
-			)
-			(justify right)
 		)
 	)
@@
 	)
 	(symbol
+		(lib_id "power:GND")
+		(at 130.81 102.87 0)
+		(unit 1)
+		(body_style 1)
+		(exclude_from_sim no)
+		(in_bom yes)
+		(on_board yes)
+		(in_pos_files yes)
+		(dnp no)
+		(property "Reference" "#PWR052"
+			(at 130.81 109.22 0)
+			(hide yes)
+			(show_name no)
+			(do_not_autoplace no)
+			(effects
+				(font
+					(size 1.27 1.27)
+				)
+			)
+		)
+		(property "Value" "GND"
+			(at 130.81 106.934 0)
+			(show_name no)
+			(do_not_autoplace no)
+			(effects
+				(font
+					(size 1.27 1.27)
+				)
+			)
+		)
+		(property "Footprint" ""
+			(at 130.81 102.87 0)
+			(hide yes)
+			(show_name no)
+			(do_not_autoplace no)
+			(effects
+				(font
+					(size 1.27 1.27)
+				)
+			)
+		)
+		(property "Datasheet" ""
+			(at 130.81 102.87 0)
+			(hide yes)
+			(show_name no)
+			(do_not_autoplace no)
+			(effects
+				(font
+					(size 1.27 1.27)
+				)
+			)
+		)
+		(property "Description" "Power symbol creates a global label with name \"GND\" , ground"
+			(at 130.81 102.87 0)
+			(hide yes)
+			(show_name no)
+			(do_not_autoplace no)
+			(effects
+				(font
+					(size 1.27 1.27)
+				)
+			)
+		)
+		(pin "1"
+		)
+		(instances
+			(project "ecvt-controller"
+				(path "/6a3c849d-efdf-47ab-8467-b82fc2fbc70f/577f7b7d-9ccb-4072-8b99-2d0e10acd900"
+					(reference "#PWR052")
+					(unit 1)
+				)
+			)
+		)
+	)
+	(symbol
 		(lib_id "Device:C")
 		(at 158.75 74.93 0)
@@
 	(symbol
 		(lib_id "Device:R")
-		(at 86.36 116.84 0)
+		(at 86.36 118.11 0)
 		(unit 1)
 		(body_style 1)
@@
 		(fields_autoplaced yes)
 		(property "Reference" "R4"
-			(at 88.9 115.5699 0)
+			(at 88.9 116.8399 0)
 			(show_name no)
 			(do_not_autoplace no)
@@
 		)
 		(property "Value" "10k"
-			(at 88.9 118.1099 0)
+			(at 88.9 119.3799 0)
 			(show_name no)
 			(do_not_autoplace no)
@@
 			)
 		)
-		(property "Footprint" ""
-			(at 84.582 116.84 90)
+		(property "Footprint" "Resistor_SMD:R_0603_1608Metric_Pad0.98x0.95mm_HandSolder"
+			(at 84.582 118.11 90)
 			(hide yes)
 			(show_name no)
@@
 		)
 		(property "Datasheet" ""
-			(at 86.36 116.84 0)
+			(at 86.36 118.11 0)
 			(hide yes)
 			(show_name no)
@@
 		)
 		(property "Description" "Resistor"
-			(at 86.36 116.84 0)
-			(hide yes)
-			(show_name no)
+			(at 86.36 118.11 0)
+			(hide yes)
+			(show_name no)

Commit message: removed old version
Connections:
- no-connect marks 0 -> 5
Changed lines of the file:
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@@
 		(color 0 0 0 0)
 	)
+	(no_connect
+		(at 69.85 116.84)
+	)
+	(no_connect
+		(at 69.85 114.3)
+	)
+	(no_connect
+		(at 69.85 109.22)
+	)
+	(no_connect
+		(at 69.85 111.76)
+	)
+	(no_connect
+		(at 69.85 119.38)
+	)
 	(wire
 		(pts
@@
 	(wire
 		(pts
+			(xy 243.84 119.38) (xy 269.24 119.38)
+		)
+		(stroke
+			(width 0)
+			(type default)
+		)
+	)
+	(wire
+		(pts
+			(xy 29.21 114.3) (xy 29.21 111.76)
+		)
+		(stroke
+			(width 0)
+			(type default)
+		)
+	)
+	(wire
+		(pts
+			(xy 176.53 100.33) (xy 176.53 99.06)
+		)
+		(stroke
+			(width 0)
+			(type default)
+		)
+	)
+	(wire
+		(pts
 			(xy 69.85 121.92) (xy 86.36 121.92)
 		)
 		(stroke
-			(width 0)
-			(type default)
-		)
-	)
-	(wire
-		(pts
-			(xy 243.84 119.38) (xy 269.24 119.38)
-		)
-		(stroke
-			(width 0)
-			(type default)
-		)
-	)
-	(wire
-		(pts
-			(xy 29.21 114.3) (xy 29.21 111.76)
-		)
-		(stroke
-			(width 0)
-			(type default)
-		)
-	)
-	(wire
-		(pts
-			(xy 176.53 100.33) (xy 176.53 99.06)
-		)
-		(stroke

Commit message: Basic ERC fixed
Parts:
- added C24: 0.1 µF, Capacitor_SMD:C_0603_1608Metric_Pad1.08x0.95mm_HandSolder, symbol Device:C
Connections:
- net +3.3V: now also C24.1
- net GND: now also C24.2; no longer U1.8 (S)
- new net S: U1.8 (S)
- no-connect marks 5 -> 6
Changed lines of the file:
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@@
 	)
 	(junction
+		(at 54.61 71.12)
+		(diameter 0)
+		(color 0 0 0 0)
+	)
+	(junction
 		(at 243.84 72.39)
 		(diameter 0)
@@
 	)
 	(no_connect
+		(at 39.37 116.84)
+	)
+	(no_connect
 		(at 69.85 111.76)
 	)
@@
 	(wire
 		(pts
+			(xy 39.37 71.12) (xy 39.37 73.66)
+		)
+		(stroke
+			(width 0)
+			(type default)
+		)
+	)
+	(wire
+		(pts
 			(xy 25.4 111.76) (xy 29.21 111.76)
 		)
@@
 	(wire
 		(pts
+			(xy 54.61 71.12) (xy 39.37 71.12)
+		)
+		(stroke
+			(width 0)
+			(type default)
+		)
+	)
+	(wire
+		(pts
 			(xy 111.76 95.25) (xy 137.16 95.25)
 		)
@@
 	(wire
 		(pts
-			(xy 54.61 76.2) (xy 54.61 86.36)
+			(xy 54.61 66.04) (xy 54.61 71.12)
 		)
 		(stroke
@@
 	(wire
 		(pts
+			(xy 54.61 71.12) (xy 54.61 86.36)
+		)
+		(stroke
+			(width 0)
+			(type default)
+		)
+	)
+	(wire
+		(pts
 			(xy 35.56 99.06) (xy 39.37 99.06)
 		)
@@
 		)
 	)
+	(hierarchical_label "S"
+		(shape input)
+		(at 130.81 102.87 180)
+		(effects
+			(font
+				(size 1.27 1.27)
+			)
+			(justify right)
+		)
+	)
 	(hierarchical_label "CS"
 		(shape input)
@@
 	)
 	(symbol
-		(lib_id "power:GND")
-		(at 130.81 102.87 0)
-		(unit 1)
-		(body_style 1)
-		(exclude_from_sim no)
-		(in_bom yes)
-		(on_board yes)
-		(in_pos_files yes)
-		(dnp no)
-		(property "Reference" "#PWR052"
-			(at 130.81 109.22 0)
-			(hide yes)
-			(show_name no)
-			(do_not_autoplace no)
-			(effects
-				(font
-					(size 1.27 1.27)
-				)
-			)
-		)
-		(property "Value" "GND"
-			(at 130.81 106.934 0)
-			(show_name no)
-			(do_not_autoplace no)
-			(effects
-				(font
-					(size 1.27 1.27)
-				)
-			)
-		)
-		(property "Footprint" ""
-			(at 130.81 102.87 0)
-			(hide yes)
-			(show_name no)
-			(do_not_autoplace no)
-			(effects
-				(font
-					(size 1.27 1.27)
-				)
-			)
-		)
-		(property "Datasheet" ""
-			(at 130.81 102.87 0)
-			(hide yes)
-			(show_name no)
-			(do_not_autoplace no)
-			(effects
-				(font
-					(size 1.27 1.27)
-				)
-			)
-		)
-		(property "Description" "Power symbol creates a global label with name \"GND\" , ground"
-			(at 130.81 102.87 0)
-			(hide yes)
-			(show_name no)
-			(do_not_autoplace no)
-			(effects
-				(font
-					(size 1.27 1.27)
-				)
-			)
-		)
-		(pin "1"
-		)
-		(instances
-			(project "ecvt-controller"
-				(path "/6a3c849d-efdf-47ab-8467-b82fc2fbc70f/577f7b7d-9ccb-4072-8b99-2d0e10acd900"
-					(reference "#PWR052")
-					(unit 1)
-				)
-			)
-		)
-	)
-	(symbol
 		(lib_id "Device:C")
 		(at 158.75 74.93 0)
@@
 	(symbol
 		(lib_id "power:+3.3V")
-		(at 54.61 76.2 0)
+		(at 54.61 66.04 0)
 		(unit 1)
 		(body_style 1)
@@
 		(fields_autoplaced yes)
 		(property "Reference" "#PWR031"
-			(at 54.61 80.01 0)
+			(at 54.61 69.85 0)
 			(hide yes)
 			(show_name no)
@@
 		)
 		(property "Value" "+3.3V"
-			(at 54.61 71.12 0)
+			(at 54.61 60.96 0)
 			(show_name no)
 			(do_not_autoplace no)
@@
 		)
 		(property "Footprint" ""
-			(at 54.61 76.2 0)
+			(at 54.61 66.04 0)
 			(hide yes)
 			(show_name no)
@@
 		)
 		(property "Datasheet" ""
-			(at 54.61 76.2 0)
+			(at 54.61 66.04 0)
 			(hide yes)
 			(show_name no)
@@
 		)
 		(property "Description" "Power symbol creates a global label with name \"+3.3V\""
-			(at 54.61 76.2 0)
+			(at 54.61 66.04 0)
 			(hide yes)
 			(show_name no)
@@
 	)
 	(symbol
+		(lib_id "power:GND")
+		(at 39.37 81.28 0)
+		(unit 1)
+		(body_style 1)
+		(exclude_from_sim no)
+		(in_bom yes)
+		(on_board yes)
+		(in_pos_files yes)
+		(dnp no)
+		(property "Reference" "#PWR053"
+			(at 39.37 87.63 0)
+			(hide yes)
+			(show_name no)
+			(do_not_autoplace no)
+			(effects
+				(font
+					(size 1.27 1.27)
+				)
+			)
+		)
+		(property "Value" "GND"
+			(at 39.37 85.09 0)
+			(show_name no)
+			(do_not_autoplace no)
+			(effects
+				(font
+					(size 1.27 1.27)
+				)
+			)
+		)
+		(property "Footprint" ""
+			(at 39.37 81.28 0)
+			(hide yes)
+			(show_name no)
+			(do_not_autoplace no)
+			(effects
+				(font
+					(size 1.27 1.27)
+				)
+			)
+		)
+		(property "Datasheet" ""
+			(at 39.37 81.28 0)
+			(hide yes)
+			(show_name no)
+			(do_not_autoplace no)
+			(effects
+				(font
+					(size 1.27 1.27)
+				)
+			)
+		)
+		(property "Description" "Power symbol creates a global label with name \"GND\" , ground"
+			(at 39.37 81.28 0)
+			(hide yes)
+			(show_name no)
+			(do_not_autoplace no)
+			(effects
+				(font
+					(size 1.27 1.27)
+				)
+			)
+		)
+		(pin "1"
+		)
+		(instances
+			(project "ecvt-controller"
+				(path "/6a3c849d-efdf-47ab-8467-b82fc2fbc70f/577f7b7d-9ccb-4072-8b99-2d0e10acd900"
+					(reference "#PWR053")
+					(unit 1)
+				)
+			)
+		)
+	)
+	(symbol
 		(lib_id "baja_symbol_library:ESD3V3AP-TP")
 		(at 186.69 91.44 0)
@@
 					(unit 1)
 				)
+			)
+		)
+	)
+	(symbol
+		(lib_id "Device:C")
+		(at 39.37 77.47 0)
+		(unit 1)
+		(body_style 1)
+		(exclude_from_sim no)
+		(in_bom yes)
+		(on_board yes)
+		(in_pos_files yes)
+		(dnp no)
+		(property "Reference" "C24"
+			(at 43.18 76.1999 0)
+			(show_name no)
+			(do_not_autoplace no)
+			(effects
+				(font
+					(size 1.27 1.27)
+				)
+				(justify left)
+			)
+		)
+		(property "Value" "0.1 µF"
+			(at 42.418 78.74 0)
+			(show_name no)
+			(do_not_autoplace no)
+			(effects
+				(font
+					(size 1.27 1.27)
+				)
+				(justify left)
+			)
+		)
+		(property "Footprint" "Capacitor_SMD:C_0603_1608Metric_Pad1.08x0.95mm_HandSolder"
+			(at 40.3352 81.28 0)
+			(hide yes)
+			(show_name no)
+			(do_not_autoplace no)
+			(effects
+				(font
+					(size 1.27 1.27)
+				)
+			)
+		)
+		(property "Datasheet" ""
+			(at 39.37 77.47 0)
+			(hide yes)
+			(show_name no)
+			(do_not_autoplace no)
+			(effects
+				(font
+					(size 1.27 1.27)
+				)
+			)
+		)
+		(property "Description" "Unpolarized capacitor"
+			(at 39.37 77.47 0)
+			(hide yes)
+			(show_name no)
+			(do_not_autoplace no)
+			(effects
+				(font
+					(size 1.27 1.27)
+				)
+			)
+		)
+		(pin "2"
+		)
+		(pin "1"
+		)
+		(instances
+			(project "ecvt-controller"
+				(path "/6a3c849d-efdf-47ab-8467-b82fc2fbc70f/577f7b7d-9ccb-4072-8b99-2d0e10acd900"
+					(reference "C24")
+					(unit 1)
+				)
