File: boards/ecvt-controller/ecvt-controller/Power.kicad_sch (KiCad schematic)
At the start: 6 parts, among them Q1 Q_PMOS, U2 TSR3-2450N

Commit message: power done
Parts:
- removed Q1: Q_PMOS, Package_TO_SOT_SMD:TO-252-2, symbol Device:Q_PMOS
- removed U2: TSR3-2450N, Converter_DCDC:Converter_DCDC_TRACO_TSR2-24xxN_TSR2-24xxxN_THT, symbol Regulator_Switching:TSR3-2450N
- added PS1: TSR_3-2450N, baja-common-parts:CONV_TSR_3-2450N, symbol TSR_3-2450N:TSR_3-2450N
- added Q1: Q_PMOS_GDS, Package_TO_SOT_SMD:TO-252-2, symbol Transistor_FET:Q_PMOS_GDS
- F1: footprint Fuse:Fuse_1206_3216Metric -> Fuse:Fuse_1206_3216Metric_Pad1.42x1.75mm_HandSolder
Connections:
- net +12V: now also Q1.2 (D)
- net +5V: now also PS1.3 (+VOUT)
- net GND: now also PS1.2 (GND)
- net at C22.2, F1.2: now also PS1.1 (+VIN)
- net at R3.1: now also Q1.1 (G)
- net at F1.1: now also Q1.3 (S)
Other:
- note removed: "D"
- note removed: "G"
- note removed: "S"
- moved on the sheet: C23
