File: boards/ecvt-controller/ecvt-controller/MCU.kicad_sch (KiCad schematic)
At the start: 1 part, among them J1 Conn_02x20_Odd_Even

Commit message: CAN actually done
Parts:
- added J2: Raspberry_Pi_2_3, symbol Connector:Raspberry_Pi_2_3
- J1: footprint (none) -> Connector_PinSocket_2.54mm:PinSocket_2x20_P2.54mm_Vertical
Connections:
- net GPIO10 renamed MOSI
- net GPIO11 renamed SCK
- net GPIO5 renamed INT
- net GPIO8 renamed CS0
- net GPIO9 renamed MISO
- new net: J2.1 (3V3), J2.17 (3V3)
- new net: J2.14 (GND), J2.20 (GND), J2.25 (GND), J2.30 (GND), J2.34 (GND), J2.39 (GND), J2.6 (GND), J2.9 (GND)
- new net: J2.2 (5V), J2.4 (5V)
Changed lines of the file:
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@@
 	(text "PIN DESCRIPTION: https://pinout.xyz/pinout/pin8_gpio14/"
 		(exclude_from_sim no)
-		(at 118.618 57.404 0)
+		(at 149.352 59.436 0)
 		(effects
 			(font
@@
 	(text "SPI0 CS0"
 		(exclude_from_sim no)
-		(at 183.896 108.458 0)
+		(at 188.468 108.966 0)
 		(effects
 			(font
@@
 	(text "SPI0 MISO"
 		(exclude_from_sim no)
-		(at 115.57 106.68 0)
+		(at 100.838 106.934 0)
 		(effects
 			(font
@@
 	(text "SPI0 CS1"
 		(exclude_from_sim no)
-		(at 183.896 110.998 0)
+		(at 188.468 111.76 0)
 		(effects
 			(font
@@
 	(text "SPI0 SCLK"
 		(exclude_from_sim no)
-		(at 115.316 109.22 0)
+		(at 100.838 109.474 0)
 		(effects
 			(font
@@
 	(text "SPI0 MOSI"
 		(exclude_from_sim no)
-		(at 115.57 103.632 0)
+		(at 101.092 103.378 0)
 		(effects
 			(font
@@
 		)
 	)
+	(hierarchical_label "MOSI"
+		(shape input)
+		(at 121.92 104.14 180)
+		(effects
+			(font
+				(size 1.27 1.27)
+			)
+			(justify right)
+		)
+	)
 	(hierarchical_label "LIMIT"
 		(shape input)
@@
 			)
 			(justify left)
+		)
+	)
+	(hierarchical_label "SCK"
+		(shape input)
+		(at 121.92 109.22 180)
+		(effects
+			(font
+				(size 1.27 1.27)
+			)
+			(justify right)
+		)
+	)
+	(hierarchical_label "INT"
+		(shape input)
+		(at 121.92 116.84 180)
+		(effects
+			(font
+				(size 1.27 1.27)
+			)
+			(justify right)
+		)
+	)
+	(hierarchical_label "CS0"
+		(shape input)
+		(at 177.8 109.22 0)
+		(effects
+			(font
+				(size 1.27 1.27)
+			)
+			(justify left)
+		)
+	)
+	(hierarchical_label "MISO"
+		(shape input)
+		(at 121.92 106.68 180)
+		(effects
+			(font
+				(size 1.27 1.27)
+			)
+			(justify right)
 		)
 	)
@@
 			)
 		)
-		(property "Footprint" ""
+		(property "Footprint" "Connector_PinSocket_2.54mm:PinSocket_2x20_P2.54mm_Vertical"
 			(at 148.59 104.14 0)
 			(hide yes)
@@
 					(unit 1)
 				)
+			)
+		)
+	)
+	(symbol
+		(lib_id "Connector:Raspberry_Pi_2_3")
+		(at 41.91 52.07 0)
+		(unit 1)
+		(body_style 1)
+		(exclude_from_sim yes)
+		(in_bom no)
+		(on_board no)
+		(in_pos_files yes)
+		(dnp no)
+		(fields_autoplaced yes)
+		(property "Reference" "J2"
+			(at 44.0533 85.09 0)
+			(show_name no)
+			(do_not_autoplace no)
+			(effects
+				(font
+					(size 1.27 1.27)
+				)
+				(justify left)
+			)
+		)
+		(property "Value" "Raspberry_Pi_2_3"
+			(at 44.0533 87.63 0)
+			(show_name no)
+			(do_not_autoplace no)
+			(effects
+				(font
+					(size 1.27 1.27)
+				)
+				(justify left)
+			)
+		)
+		(property "Footprint" ""
+			(at 41.91 52.07 0)
+			(hide yes)
+			(show_name no)
+			(do_not_autoplace no)
+			(effects
+				(font
+					(size 1.27 1.27)
+				)
+			)
+		)
+		(property "Datasheet" "https://www.raspberrypi.org/documentation/hardware/raspberrypi/schematics/rpi_SCH_3bplus_1p0_reduced.pdf"
+			(at 102.87 96.52 0)
+			(hide yes)
+			(show_name no)
+			(do_not_autoplace no)
+			(effects
+				(font
+					(size 1.27 1.27)
+				)
+			)
+		)
+		(property "Description" "expansion header for Raspberry Pi 2 & 3"
+			(at 41.91 52.07 0)
+			(hide yes)
+			(show_name no)
+			(do_not_autoplace no)
+			(effects
+				(font
+					(size 1.27 1.27)
+				)
+			)
+		)
+		(pin "20"
+		)
+		(pin "7"
+		)
+		(pin "25"
+		)
+		(pin "27"
+		)
+		(pin "2"
+		)
+		(pin "4"
+		)
+		(pin "1"
+		)
+		(pin "3"
+		)
+		(pin "5"
+		)
+		(pin "9"
+		)
+		(pin "10"
+		)
+		(pin "11"
+		)
+		(pin "12"
+		)
+		(pin "6"
+		)
+		(pin "13"
+		)
+		(pin "16"
+		)
+		(pin "14"
+		)
+		(pin "17"
+		)
+		(pin "19"
+		)
+		(pin "21"
+		)
+		(pin "22"
+		)
+		(pin "15"
+		)
+		(pin "8"
+		)
+		(pin "18"
+		)
+		(pin "23"
+		)
+		(pin "24"
+		)
+		(pin "26"
+		)
+		(pin "38"
+		)
+		(pin "37"
+		)
+		(pin "40"
+		)
+		(pin "32"
+		)
+		(pin "29"
+		)
+		(pin "31"
+		)
+		(pin "36"
+		)
+		(pin "39"
+		)
+		(pin "28"
+		)
+		(pin "30"
+		)
+		(pin "35"
+		)
+		(pin "33"
+		)
+		(pin "34"
+		)
+		(instances
+			(project "ecvt-controller"
+				(path "/6a3c849d-efdf-47ab-8467-b82fc2fbc70f/86d3e2f6-ea24-425a-b24f-155dc33c446a"
+					(reference "J2")
+					(unit 1)
+				)

Commit message: almost done schmatic
Parts:
- added H1, H2, H3, H4: MountingHole, MountingHole:MountingHole_2.7mm_M2.5, symbol Mechanical:MountingHole
Connections:
- net GPIO6 renamed S
Other:
- note added: "DR Decisions - How many open pins / 5V - Analog?"

Commit message: components done. RAHHHHH
Parts:
- added C12: 4.7µF, Capacitor_SMD:C_0603_1608Metric_Pad1.08x0.95mm_HandSolder, symbol Device:C
- added C13, C14: 0.1 µF, Capacitor_SMD:C_0603_1608Metric_Pad1.08x0.95mm_HandSolder, symbol Device:C
Connections:
- net +3.3V: now also C14.1
- net +5V: now also C12.1, C13.1
- net GND: now also C12.2, C13.2, C14.2

Commit message: Pre-DR
Connections:
- net GPIO17 is gone; now on net PRIMARY_HALL: J1.11 (Pin_11)
- net GPIO22 is gone; now on net LIMIT: J1.15 (Pin_15)
- net GPIO27 is gone; now on net SECONDARY_HALL: J1.13 (Pin_13)
- net LIMIT: no longer J1.22 (Pin_22)
- net PRIMARY_HALL: no longer J1.16 (Pin_16)
- net SECONDARY_HALL: no longer J1.18 (Pin_18)
- new net GPIO23: J1.16 (Pin_16)
- new net GPIO24: J1.18 (Pin_18)
- new net GPIO25: J1.22 (Pin_22)
Changed lines of the file:
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@@
 	(hierarchical_label "LIMIT"
 		(shape input)
-		(at 196.85 106.68 0)
+		(at 121.92 99.06 180)
 		(effects
 			(font
 				(size 1.27 1.27)
 			)
-			(justify left)
+			(justify right)
+		)
+	)
+	(hierarchical_label "PRIMARY_HALL"
+		(shape input)
+		(at 121.92 93.98 180)
+		(effects
+			(font
+				(size 1.27 1.27)
+			)
+			(justify right)
 		)
 	)
 	(hierarchical_label "SECONDARY_HALL"
 		(shape input)
-		(at 196.85 101.6 0)
+		(at 121.92 96.52 180)
 		(effects
 			(font
 				(size 1.27 1.27)
 			)
-			(justify left)
+			(justify right)
 		)
 	)
@@
 		)
 	)
-	(hierarchical_label "PRIMARY_HALL"
-		(shape input)
-		(at 196.85 99.06 0)
-		(effects
-			(font
-				(size 1.27 1.27)
-			)
-			(justify left)
-		)
-	)

Commit message: removed old version
Changed lines of the file:
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@@
+	)
+	(junction
+		(at 125.73 63.5)
+		(diameter 0)
+		(color 0 0 0 0)
 	)
 	(junction
@@
 	(wire
 		(pts
+			(xy 125.73 63.5) (xy 129.54 63.5)
+		)
+		(stroke
+			(width 0)
+			(type default)
+		)
+	)
+	(wire
+		(pts
 			(xy 156.21 91.44) (xy 177.8 91.44)
 		)
@@
 	(wire
 		(pts
-			(xy 116.84 63.5) (xy 129.54 63.5)
+			(xy 116.84 63.5) (xy 125.73 63.5)
 		)
 		(stroke
@@
 					(unit 1)
 				)
+			)
+		)
+	)
+	(symbol
+		(lib_id "power:PWR_FLAG")
+		(at 125.73 63.5 0)
+		(unit 1)
+		(body_style 1)
+		(exclude_from_sim no)
+		(in_bom yes)
+		(on_board yes)
+		(in_pos_files yes)
+		(dnp no)
+		(fields_autoplaced yes)
+		(property "Reference" "#FLG05"
+			(at 125.73 61.595 0)
+			(hide yes)
+			(show_name no)
+			(do_not_autoplace no)
+			(effects
+				(font
+					(size 1.27 1.27)
+				)
+			)
+		)
+		(property "Value" "PWR_FLAG"
+			(at 125.73 58.42 0)
+			(show_name no)
+			(do_not_autoplace no)
+			(effects
+				(font
+					(size 1.27 1.27)
+				)
+			)
+		)
+		(property "Footprint" ""
+			(at 125.73 63.5 0)
+			(hide yes)
+			(show_name no)
+			(do_not_autoplace no)
+			(effects
+				(font
+					(size 1.27 1.27)
+				)
+			)
+		)
+		(property "Datasheet" ""
+			(at 125.73 63.5 0)
+			(hide yes)
+			(show_name no)
+			(do_not_autoplace no)
+			(effects
+				(font
+					(size 1.27 1.27)
+				)
+			)
+		)
+		(property "Description" "Special symbol for telling ERC where power comes from"
+			(at 125.73 63.5 0)
+			(hide yes)
+			(show_name no)
+			(do_not_autoplace no)
+			(effects
+				(font
+					(size 1.27 1.27)
+				)
+			)
+		)
+		(pin "1"
+		)
+		(instances
+			(project "ecvt-controller"
+				(path "/6a3c849d-efdf-47ab-8467-b82fc2fbc70f/86d3e2f6-ea24-425a-b24f-155dc33c446a"
+					(reference "#FLG05")
+					(unit 1)
+				)

Commit message: Basic ERC fixed
Parts:
- removed J2: Raspberry_Pi_2_3, symbol Connector:Raspberry_Pi_2_3
Connections:
- net GPIO0: no longer names the net of J1.27 (Pin_27)
- net GPIO1: no longer names the net of J1.28 (Pin_28)
- net GPIO12: no longer names the net of J1.32 (Pin_32)
- net GPIO13: no longer names the net of J1.33 (Pin_33)
- net GPIO14: no longer names the net of J1.8 (Pin_8)
- net GPIO15: no longer names the net of J1.10 (Pin_10)
- net GPIO16: no longer names the net of J1.36 (Pin_36)
- net GPIO18: no longer names the net of J1.12 (Pin_12)
- net GPIO19 renamed Sig1
- net GPIO2: no longer names the net of J1.3 (Pin_3)
- net GPIO20: no longer names the net of J1.38 (Pin_38)
- net GPIO21: no longer names the net of J1.40 (Pin_40)
- net GPIO23: no longer names the net of J1.16 (Pin_16)
- net GPIO24: no longer names the net of J1.18 (Pin_18)
- net GPIO25: no longer names the net of J1.22 (Pin_22)
- net GPIO26 renamed Sig2
- net GPIO3: no longer names the net of J1.5 (Pin_5)
- net GPIO4: no longer names the net of J1.7 (Pin_7)
- net GPIO7: no longer names the net of J1.26 (Pin_26)
- net LIMIT renamed Limit
- net PRIMARY_HALL renamed Primary
- net SECONDARY_HALL renamed Secondary
- no-connect marks 0 -> 17
Other:
- note added: "GPIO0"
- note added: "GPIO1"
- note added: "GPIO10"
- note added: "GPIO11"
- note added: "GPIO12"
- note added: "GPIO13"
- note added: "GPIO14"
- note added: "GPIO15"
- note added: "GPIO16"
- note added: "GPIO17"
- note added: "GPIO18"
- note added: "GPIO19"
- note added: "GPIO2"
- note added: "GPIO20"
- note added: "GPIO21"
- note added: "GPIO22"
- note added: "GPIO23"
- note added: "GPIO24"
- note added: "GPIO25"
- note added: "GPIO26"
- note added: "GPIO27"
- note added: "GPIO3"
- note added: "GPIO4"
- note added: "GPIO5"
- note added: "GPIO6"
- note added: "GPIO7"
- note added: "GPIO8"
- note added: "GPIO9"
- note removed: "DR Decisions - How many open pins / 5V - Analog?"

Commit message: ADC done
Connections:
- net SDA: now reaches J1.3 (Pin_3)
- net SCL: now reaches J1.5 (Pin_5)
- no-connect marks 17 -> 15
Changed lines of the file:
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@@
 	(text "I2C clock: fixed 1.8k pull up to 3.3V\n"
 		(exclude_from_sim no)
-		(at 102.87 85.852 0)
+		(at 101.346 88.392 0)
 		(effects
 			(font
@@
 	(text "12C data: fixed 1.8k pull up to 3.3V\n"
 		(exclude_from_sim no)
-		(at 103.124 83.566 0)
+		(at 103.886 80.518 0)
 		(effects
 			(font
@@
 	)
 	(no_connect
-		(at 121.92 83.82)
-	)
-	(no_connect
 		(at 177.8 127)
 	)
@@
 	(no_connect
 		(at 121.92 114.3)
-	)
-	(no_connect
-		(at 121.92 86.36)
 	)
 	(wire
@@
 		)
 	)
+	(hierarchical_label "SCL"
+		(shape input)
+		(at 121.92 86.36 180)
+		(effects
+			(font
+				(size 1.27 1.27)
+			)
+			(justify right)
+		)
+	)
 	(hierarchical_label "Sig1"
 		(shape input)
@@
 		(effects
 			(font
+				(size 1.27 1.27)
+			)
+			(justify right)
+		)
+	)
+	(hierarchical_label "SDA"
+		(shape input)
+		(at 121.92 83.82 180)
+		(effects
+			(font

Commit message: Capacitors !!!!
Parts:
- removed C12: 4.7µF, Capacitor_SMD:C_0603_1608Metric_Pad1.08x0.95mm_HandSolder, symbol Device:C
- removed C13, C14: 0.1 µF, Capacitor_SMD:C_0603_1608Metric_Pad1.08x0.95mm_HandSolder, symbol Device:C
- added C3: 4.7µF, Capacitor_SMD:C_0805_2012Metric_Pad1.18x1.45mm_HandSolder, symbol baja-common-parts:C_0805
- added C4, C5: 0.1 µF, Capacitor_SMD:C_0603_1608Metric_Pad1.08x0.95mm_HandSolder, symbol baja-common-parts:C_0603
Connections:
- net +3.3V: now also C4.1
- net +5V: now also C3.1, C5.1
- net GND: now also C3.2, C4.2, C5.2
