File: boards/ecvt-controller/ecvt-controller/MCU.kicad_sch (KiCad schematic)
At the start: 8 parts, among them J1 Conn_02x20_Odd_Even

Commit message: Done  danadan done done da da
Connections:
- net +3.3V: no longer J1.17 (Pin_17)
- net S: no longer names the net of J1.31 (Pin_31)
- new net +3.3V(v2): J1.17 (Pin_17)
- no-connect marks 15 -> 16
Changed lines of the file:
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@@
+	)
+	(no_connect
+		(at 121.92 119.38)
 	)
 	(no_connect
@@
 		(shape input)
 		(at 121.92 109.22 180)
-		(effects
-			(font
-				(size 1.27 1.27)
-			)
-			(justify right)
-		)
-	)
-	(hierarchical_label "S"
-		(shape input)
-		(at 121.92 119.38 180)
 		(effects
 			(font
@@
 			)
 		)
-		(property "Value" "+3.3V"
+		(property "Value" "+3.3V(v2)"
 			(at 134.62 101.5999 90)
 			(show_name no)
