File: boards/ecvt-controller/ecvt-controller/ADC.kicad_sch (KiCad schematic)
At the start: 6 parts, among them U2 ADS1115IDGS

Commit message: Capacitors !!!!
Parts:
- removed C3: 0.1uF, Capacitor_SMD:C_0603_1608Metric_Pad1.08x0.95mm_HandSolder, symbol baja-common-parts:C_0603
- added C13: 0.1 µF, Capacitor_SMD:C_0603_1608Metric_Pad1.08x0.95mm_HandSolder, symbol baja-common-parts:C_0603
Connections:
- net +3.3V: now also C13.1
- net GND: now also C13.2
