File: boards/ecvt-controller/ecvt-controller/ADC.kicad_sch (KiCad schematic)
At the start: 6 parts, among them U2 ADS1115IDGS

Commit message: Rough Placement
no traces, slightly worries about 5V and 3.3V
Connections:
- net AIN0: now also R1.2, R2.1, U2.4 (AIN0)
- net AIN1: now also R8.2, R9.1, U2.5 (AIN1)
Changed lines of the file:
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@@
+		)
+	)
+	(label "AIN1"
+		(at 120.65 90.17 0)
+		(effects
+			(font
+				(size 1.27 1.27)
+			)
+			(justify left bottom)
+		)
+	)
+	(label "AIN0"
+		(at 120.65 87.63 0)
+		(effects
+			(font
+				(size 1.27 1.27)
+			)
+			(justify left bottom)
 		)
 	)

Commit message: Done  danadan done done da da
Connections:
- net AIN0: no longer R1.2, R2.1, U2.4 (AIN0)
- net AIN1: no longer R8.2, R9.1, U2.5 (AIN1)
- new net AIN0_in: R1.2, R2.1, U2.4 (AIN0)
- new net AIN1_in: R8.2, R9.1, U2.5 (AIN1)
Changed lines of the file:
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@@
 		)
 	)
-	(label "AIN1"
+	(label "AIN1_in"
 		(at 120.65 90.17 0)
 		(effects
@@
 		)
 	)
-	(label "AIN0"
+	(label "AIN0_in"
 		(at 120.65 87.63 0)
 		(effects
