File: boards/ecvt-controller/ecvt-controller/Connectors.kicad_sch (KiCad schematic)
At the start: 4 parts, among them J3 1720420206, J4 1720420206, J5 917786-1, J6 917780-1

Commit message: cap sizing
Parts:
- J3, J4: footprint 1720420206:CONN_SD-172042-001_02_BL_MOL -> Molex_SuperSabre:CONN_SD-172042-001_02_BL_MOL
Changed lines of the file:
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@@
 			)
 		)
-		(property "Footprint" "1720420206:CONN_SD-172042-001_02_BL_MOL"
+		(property "Footprint" "Molex_SuperSabre:CONN_SD-172042-001_02_BL_MOL"
 			(at 152.4 68.58 0)
 			(hide yes)
@@
 			)
 		)
-		(property "Footprint" "1720420206:CONN_SD-172042-001_02_BL_MOL"
+		(property "Footprint" "Molex_SuperSabre:CONN_SD-172042-001_02_BL_MOL"
 			(at 142.24 100.33 0)
 			(hide yes)

Commit message: components done. RAHHHHH
Parts:
- added D6, D7, D8: DF2S5M4CTL3FCT-ND, Diode_SMD:D_SOD-882, symbol Device:D_Zener
Connections:
- net GND: now also D6.2 (A), D7.2 (A), D8.2 (A)
- net Limit: now also D8.1 (K)
- net Primary: now also D6.1 (K)
- net Secondary: now also D7.1 (K)

Commit message: Pre-DR
Parts:
- removed J4: 1720420206, Molex_SuperSabre:CONN_SD-172042-001_02_BL_MOL, symbol 1720420206:1720420206
Other:
- note removed: "Motor"
Changed lines of the file:
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@@
-		)
-	)
-	(text "Motor\n"
-		(exclude_from_sim no)
-		(at 151.13 94.742 0)
-		(effects
-			(font
-				(size 1.27 1.27)
-			)
 		)
 	)
@@
 	(wire
 		(pts
-			(xy 139.7 102.87) (xy 142.24 102.87)
-		)
-		(stroke
-			(width 0)
-			(type default)
-		)
-	)
-	(wire
-		(pts
 			(xy 73.66 72.39) (xy 73.66 76.2)
 		)
@@
 	(wire
 		(pts
-			(xy 139.7 102.87) (xy 139.7 104.14)
-		)
-		(stroke
-			(width 0)
-			(type default)
-		)
-	)
-	(wire
-		(pts
 			(xy 72.39 64.77) (xy 72.39 66.04)
 		)
@@
 	(wire
 		(pts
-			(xy 139.7 97.79) (xy 139.7 100.33)
-		)
-		(stroke
-			(width 0)
-			(type default)
-		)
-	)
-	(wire
-		(pts
 			(xy 69.85 64.77) (xy 72.39 64.77)
 		)
@@
 		(pts
 			(xy 69.85 72.39) (xy 73.66 72.39)
-		)
-		(stroke
-			(width 0)
-			(type default)
-		)
-	)
-	(wire
-		(pts
-			(xy 139.7 100.33) (xy 142.24 100.33)
 		)
 		(stroke
@@
 		)
 	)
-	(hierarchical_label "12V_Motor_Driver"
-		(shape input)
-		(at 139.7 97.79 180)
-		(effects
-			(font
-				(size 1.27 1.27)
-			)
-			(justify right)
-		)
-	)
 	(hierarchical_label "Limit"
 		(shape input)
@@
 	)
 	(symbol
-		(lib_id "1720420206:1720420206")
-		(at 142.24 100.33 0)
-		(unit 1)
-		(body_style 1)
-		(exclude_from_sim no)
-		(in_bom yes)
-		(on_board yes)
-		(in_pos_files yes)
-		(dnp no)
-		(fields_autoplaced yes)
-		(property "Reference" "J4"
-			(at 156.21 100.3299 0)
-			(show_name no)
-			(do_not_autoplace no)
-			(effects
-				(font
-					(size 1.27 1.27)
-				)
-				(justify left)
-			)
-		)
-		(property "Value" "1720420206"
-			(at 156.21 102.8699 0)
-			(show_name no)
-			(do_not_autoplace no)
-			(effects
-				(font
-					(size 1.27 1.27)
-				)
-				(justify left)
-			)
-		)
-		(property "Footprint" "Molex_SuperSabre:CONN_SD-172042-001_02_BL_MOL"
-			(at 142.24 100.33 0)
-			(hide yes)
-			(show_name no)
-			(do_not_autoplace no)
-			(effects
-				(font
-					(size 1.27 1.27)
-				)
-				(justify bottom)
-			)
-		)
-		(property "Datasheet" "https://www.molex.com/en-us/products/part-detail-pdf/1720420206?display=pdf"
-			(at 142.24 100.33 0)
-			(hide yes)
-			(show_name no)
-			(do_not_autoplace no)
-			(effects
-				(font
-					(size 1.27 1.27)
-				)
-				(justify bottom)
-			)
-		)
-		(property "Description" "Super Sabre Vertical Header, 7.50mm Pitch, 2 Circuits, Glow-Wire Capable, 5.33mm Tail Length, with Board Lock, Complies with UL1977 Finger Proof Standards"
-			(at 142.24 100.33 0)
-			(hide yes)
-			(show_name no)
-			(do_not_autoplace no)
-			(effects
-				(font
-					(size 1.27 1.27)
-				)
-				(justify bottom)
-			)
-		)
-		(property "MFR_NAME" "Molex"
-			(at 142.24 100.33 0)
-			(hide yes)
-			(show_name no)
-			(do_not_autoplace no)
-			(effects
-				(font
-					(size 1.27 1.27)
-				)
-				(justify bottom)
-			)
-		)
-		(property "MANUFACTURER_PART_NUMBER" "1720420206"
-			(at 142.24 100.33 0)
-			(hide yes)
-			(show_name no)
-			(do_not_autoplace no)
-			(effects
-				(font
-					(size 1.27 1.27)
-				)
-				(justify bottom)
-			)
-		)
-		(pin "1"
-		)
-		(pin "2"
-		)
-		(instances
-			(project "ecvt-controller"
-				(path "/6a3c849d-efdf-47ab-8467-b82fc2fbc70f/2eb35e44-f3d1-4b8a-b6ba-ac006b5b3fd5"
-					(reference "J4")
-					(unit 1)
-				)
-			)
-		)
-	)
-	(symbol
 		(lib_id "power:GND")
 		(at 86.36 77.47 270)
@@
 					(unit 1)
 				)
-			)
-		)
-	)
-	(symbol
-		(lib_id "power:GND")
-		(at 139.7 104.14 0)
-		(unit 1)
-		(body_style 1)
-		(exclude_from_sim no)
-		(in_bom yes)
-		(on_board yes)
-		(in_pos_files yes)
-		(dnp no)
-		(property "Reference" "#PWR041"
-			(at 139.7 110.49 0)
-			(hide yes)
-			(show_name no)
-			(do_not_autoplace no)
-			(effects
-				(font
-					(size 1.27 1.27)
-				)
-			)
-		)
-		(property "Value" "GND"
-			(at 139.7 108.204 0)
-			(show_name no)
-			(do_not_autoplace no)
-			(effects
-				(font
-					(size 1.27 1.27)
-				)
-			)
-		)
-		(property "Footprint" ""
-			(at 139.7 104.14 0)
-			(hide yes)
-			(show_name no)
-			(do_not_autoplace no)
-			(effects
-				(font
-					(size 1.27 1.27)
-				)
-			)
-		)
-		(property "Datasheet" ""
-			(at 139.7 104.14 0)
-			(hide yes)
-			(show_name no)
-			(do_not_autoplace no)
-			(effects
-				(font
-					(size 1.27 1.27)
-				)
-			)
-		)
-		(property "Description" "Power symbol creates a global label with name \"GND\" , ground"
-			(at 139.7 104.14 0)
-			(hide yes)
-			(show_name no)
-			(do_not_autoplace no)
-			(effects
-				(font
-					(size 1.27 1.27)
-				)
-			)
-		)
-		(pin "1"
-		)
-		(instances
-			(project "ecvt-controller"
-				(path "/6a3c849d-efdf-47ab-8467-b82fc2fbc70f/2eb35e44-f3d1-4b8a-b6ba-ac006b5b3fd5"
-					(reference "#PWR041")
-					(unit 1)
-				)

Commit message: removed old version
Parts:
- removed J3: 1720420206, Molex_SuperSabre:CONN_SD-172042-001_02_BL_MOL, symbol 1720420206:1720420206
- added J4: 15311026, baja_footprint_library:MOLEX_15311026, symbol baja_symbol_library:15311026
Connections:
- net +12V: now also J4.1
- net GND: now also J4.2

Commit message: Basic ERC fixed
Parts:
- added J3: 917782-1, baja-common-parts:CON4_1X4_P100, symbol baja-common-parts:917782-1
Connections:
- net +3.3V: now also J3.1
- net GND: now also J3.4
- new net Sig1: J3.2
- new net Sig2: J3.3

Commit message: ADC done
Parts:
- added J2: 917782-1, baja-common-parts:CON4_1X4_P100, symbol baja-common-parts:917782-1
Connections:
- net GND: now also J2.4
- new net +5V: J2.1
- new net AIN0: J2.2
- new net AIN1: J2.3

Commit message: almost there
Parts:
- removed D6, D7, D8: DF2S5M4CTL3FCT-ND, Diode_SMD:D_SOD-882, symbol Device:D_Zener
- added D2, D3, D4, D5, D6, D7, D8: D_TVS, Diode_SMD:D_SOD-323_HandSoldering, symbol Device:D_TVS
Connections:
- net AIN0: now also D7.2 (A2)
- net AIN1: now also D8.2 (A2)
- net GND: now also D2.1 (A1), D3.1 (A1), D4.1 (A1), D5.1 (A1), D6.1 (A1), D7.1 (A1), D8.1 (A1)
- net Limit: now also D4.2 (A2)
- net Primary: now also D2.2 (A2)
- net Secondary: now also D3.2 (A2)
- net Sig1: now also D5.2 (A2)
- net Sig2: now also D6.2 (A2)
Other:
- moved on the sheet: J2, J6
