File: boards/ecvt-controller/ecvt-controller/Connectors.kicad_sch (KiCad schematic)
At the start: 12 parts, among them J2 917782-1, J3 917782-1, J4 15311026, J5 917786-1, J6 917780-1

Commit message: Rough Placement
no traces, slightly worries about 5V and 3.3V
Connections:
- net AIN0: now also D8.2 (A2), J2.3; no longer D7.2 (A2), J2.2
- net AIN1: now also D7.2 (A2), J2.2; no longer D8.2 (A2), J2.3
- net Sig1: now also D6.2 (A2), J3.3; no longer D5.2 (A2), J3.2
- net Sig2: now also D5.2 (A2), J3.2; no longer D6.2 (A2), J3.3
Changed lines of the file:
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@@
 	(hierarchical_label "Sig1"
 		(shape input)
-		(at 127 95.25 180)
+		(at 127 97.79 180)
+		(effects
+			(font
+				(size 1.27 1.27)
+			)
+			(justify right)
+		)
+	)
+	(hierarchical_label "AIN1"
+		(shape input)
+		(at 127 134.62 180)
 		(effects
 			(font
@@
 	(hierarchical_label "Sig2"
 		(shape input)
-		(at 127 97.79 180)
+		(at 127 95.25 180)
 		(effects
 			(font
@@
 	(hierarchical_label "AIN0"
 		(shape input)
-		(at 127 134.62 180)
+		(at 127 137.16 180)
 		(effects
 			(font
@@
 		(effects
 			(font
-				(size 1.27 1.27)
-			)
-			(justify right)
-		)
-	)
-	(hierarchical_label "AIN1"
-		(shape input)
-		(at 127 137.16 180)
-		(effects
-			(font

Commit message: Done  danadan done done da da
Changed lines of the file:
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@@
+	)
+	(junction
+		(at 128.27 97.79)
+		(diameter 0)
+		(color 0 0 0 0)
 	)
 	(junction
@@
 	)
 	(junction
-		(at 128.27 97.79)
-		(diameter 0)
-		(color 0 0 0 0)
-	)
-	(junction
 		(at 129.54 137.16)
 		(diameter 0)
@@
 	(wire
 		(pts
-			(xy 127 97.79) (xy 128.27 97.79)
+			(xy 123.19 97.79) (xy 128.27 97.79)
 		)
 		(stroke
@@
 	(wire
 		(pts
-			(xy 127 95.25) (xy 128.27 95.25)
+			(xy 123.19 95.25) (xy 128.27 95.25)
 		)
 		(stroke
@@
 	(hierarchical_label "Sig1"
 		(shape input)
-		(at 127 97.79 180)
+		(at 123.19 97.79 180)
 		(effects
 			(font
@@
 	(hierarchical_label "Sig2"
 		(shape input)
-		(at 127 95.25 180)
+		(at 123.19 95.25 180)
 		(effects
 			(font
