File: boards/ecvt-controller/ecvt-controller/ecvt-controller.kicad_sch (KiCad schematic)
At the start: 0 parts

Commit message: CAN actually done
Other:
- sheet CAN ports: added CANH, CANL, CS, INT, S, SCK, SI, SO; removed none
- sheet MCU ports: added CS0, INT, LIMIT, MISO, MOSI, SCK; removed LIMIT/LIN_POT
Changed lines of the file:
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@@
 	(generator_version "10.0")
 	(paper "A4")
+	(wire
+		(pts
+			(xy 158.75 72.39) (xy 158.75 92.71)
+		)
+		(stroke
+			(width 0)
+			(type default)
+		)
+	)
+	(wire
+		(pts
+			(xy 147.32 72.39) (xy 147.32 92.71)
+		)
+		(stroke
+			(width 0)
+			(type default)
+		)
+	)
+	(wire
+		(pts
+			(xy 161.29 72.39) (xy 161.29 92.71)
+		)
+		(stroke
+			(width 0)
+			(type default)
+		)
+	)
+	(wire
+		(pts
+			(xy 166.37 72.39) (xy 166.37 92.71)
+		)
+		(stroke
+			(width 0)
+			(type default)
+		)
+	)
+	(wire
+		(pts
+			(xy 153.67 72.39) (xy 153.67 92.71)
+		)
+		(stroke
+			(width 0)
+			(type default)
+		)
+	)
 	(sheet
 		(at 128.27 92.71)
@@
 			)
 		)
+		(pin "S" input
+			(at 133.35 92.71 90)
+			(effects
+				(font
+					(size 1.27 1.27)
+				)
+				(justify right)
+			)
+		)
+		(pin "CANH" input
+			(at 151.13 119.38 270)
+			(effects
+				(font
+					(size 1.27 1.27)
+				)
+				(justify left)
+			)
+		)
+		(pin "CANL" input
+			(at 157.48 119.38 270)
+			(effects
+				(font
+					(size 1.27 1.27)
+				)
+				(justify left)
+			)
+		)
+		(pin "INT" input
+			(at 147.32 92.71 90)
+			(effects
+				(font
+					(size 1.27 1.27)
+				)
+				(justify right)
+			)
+		)
+		(pin "CS" input
+			(at 153.67 92.71 90)
+			(effects
+				(font
+					(size 1.27 1.27)
+				)
+				(justify right)
+			)
+		)
+		(pin "SI" input
+			(at 158.75 92.71 90)
+			(effects
+				(font
+					(size 1.27 1.27)
+				)
+				(justify right)
+			)
+		)
+		(pin "SO" input
+			(at 161.29 92.71 90)
+			(effects
+				(font
+					(size 1.27 1.27)
+				)
+				(justify right)
+			)
+		)
+		(pin "SCK" input
+			(at 166.37 92.71 90)
+			(effects
+				(font
+					(size 1.27 1.27)
+				)
+				(justify right)
+			)
+		)
 		(instances
 			(project "ecvt-controller"
@@
 			)
 		)
-		(pin "LIMIT{slash}LIN_POT" input
+		(pin "PRIMARY_HALL" input
+			(at 147.32 43.18 90)
+			(effects
+				(font
+					(size 1.27 1.27)
+				)
+				(justify right)
+			)
+		)
+		(pin "SECONDARY_HALL" input
+			(at 157.48 43.18 90)
+			(effects
+				(font
+					(size 1.27 1.27)
+				)
+				(justify right)
+			)
+		)
+		(pin "LIMIT" input
+			(at 138.43 43.18 90)
+			(effects
+				(font
+					(size 1.27 1.27)
+				)
+				(justify right)
+			)
+		)
+		(pin "CS0" input
 			(at 153.67 72.39 270)
 			(effects
@@
 			)
 		)
-		(pin "PRIMARY_HALL" input
+		(pin "MOSI" input
 			(at 158.75 72.39 270)
 			(effects
@@
 			)
 		)
-		(pin "SECONDARY_HALL" input
-			(at 163.83 72.39 270)
-			(effects
-				(font
+		(pin "INT" input
+			(at 147.32 72.39 270)
+			(effects
+				(font
+					(size 1.27 1.27)
+				)
+				(justify left)
+			)
+		)
+		(pin "SCK" input
+			(at 166.37 72.39 270)
+			(effects
+				(font
+					(size 1.27 1.27)
+				)
+				(justify left)
+			)
+		)
+		(pin "MISO" input
+			(at 161.29 72.39 270)
+			(effects
+				(font

Commit message: almost done schmatic
Other:
- added sheet Connectors (Connectors.kicad_sch)
- sheet MCU ports: added S; removed none
Changed lines of the file:
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@@
+	(wire
+		(pts
+			(xy 220.98 104.14) (xy 228.6 104.14)
+		)
+		(stroke
+			(width 0)
+			(type default)
+		)
+	)
+	(wire
+		(pts
+			(xy 172.72 60.96) (xy 193.04 60.96)
+		)
+		(stroke
+			(width 0)
+			(type default)
+		)
+	)
+	(wire
+		(pts
+			(xy 172.72 57.15) (xy 196.85 57.15)
+		)
+		(stroke
+			(width 0)
+			(type default)
+		)
+	)
+	(wire
+		(pts
+			(xy 196.85 57.15) (xy 196.85 91.44)
+		)
+		(stroke
+			(width 0)
+			(type default)
+		)
+	)
+	(wire
+		(pts
+			(xy 200.66 53.34) (xy 200.66 91.44)
+		)
+		(stroke
+			(width 0)
+			(type default)
+		)
+	)
+	(wire
+		(pts
+			(xy 172.72 53.34) (xy 200.66 53.34)
+		)
+		(stroke
+			(width 0)
+			(type default)
+		)
+	)
 	(wire
 		(pts
@@
 	(wire
 		(pts
+			(xy 173.99 102.87) (xy 181.61 102.87)
+		)
+		(stroke
+			(width 0)
+			(type default)
+		)
+	)
+	(wire
+		(pts
+			(xy 173.99 109.22) (xy 181.61 109.22)
+		)
+		(stroke
+			(width 0)
+			(type default)
+		)
+	)
+	(wire
+		(pts
 			(xy 161.29 72.39) (xy 161.29 92.71)
 		)
@@
 	(wire
 		(pts
+			(xy 193.04 60.96) (xy 193.04 91.44)
+		)
+		(stroke
+			(width 0)
+			(type default)
+		)
+	)
+	(wire
+		(pts
 			(xy 166.37 72.39) (xy 166.37 92.71)
 		)
@@
 			(width 0)
 			(type default)
+		)
+	)
+	(sheet
+		(at 181.61 91.44)
+		(size 39.37 27.94)
+		(exclude_from_sim no)
+		(in_bom yes)
+		(on_board yes)
+		(dnp no)
+		(fields_autoplaced yes)
+		(stroke
+			(width 0.1524)
+			(type solid)
+		)
+		(fill
+			(color 0 0 0 0)
+		)
+		(property "Sheetname" "Connectors"
+			(at 181.61 90.7284 0)
+			(show_name no)
+			(do_not_autoplace no)
+			(effects
+				(font
+					(size 1.27 1.27)
+				)
+				(justify left bottom)
+			)
+		)
+		(property "Sheetfile" "Connectors.kicad_sch"
+			(at 181.61 119.9646 0)
+			(show_name no)
+			(do_not_autoplace no)
+			(effects
+				(font
+					(size 1.27 1.27)
+				)
+				(justify left top)
+			)
+		)
+		(pin "12V_Motor_Driver" input
+			(at 220.98 104.14 0)
+			(effects
+				(font
+					(size 1.27 1.27)
+				)
+				(justify right)
+			)
+		)
+		(pin "CANL" input
+			(at 181.61 102.87 180)
+			(effects
+				(font
+					(size 1.27 1.27)
+				)
+				(justify left)
+			)
+		)
+		(pin "CANH" input
+			(at 181.61 109.22 180)
+			(effects
+				(font
+					(size 1.27 1.27)
+				)
+				(justify left)
+			)
+		)
+		(pin "Limit" input
+			(at 200.66 91.44 90)
+			(effects
+				(font
+					(size 1.27 1.27)
+				)
+				(justify right)
+			)
+		)
+		(pin "Primary" input
+			(at 196.85 91.44 90)
+			(effects
+				(font
+					(size 1.27 1.27)
+				)
+				(justify right)
+			)
+		)
+		(pin "Secondary" input
+			(at 193.04 91.44 90)
+			(effects
+				(font
+					(size 1.27 1.27)
+				)
+				(justify right)
+			)
+		)
+		(instances
+			(project "ecvt-controller"
+				(path "/6a3c849d-efdf-47ab-8467-b82fc2fbc70f"
+					(page "5")
+				)
+			)
 		)
 	)
@@
 		)
 		(pin "S" input
-			(at 133.35 92.71 90)
+			(at 139.7 92.71 90)
 			(effects
 				(font
@@
 		)
 		(pin "CANH" input
-			(at 151.13 119.38 270)
-			(effects
-				(font
-					(size 1.27 1.27)
-				)
-				(justify left)
+			(at 173.99 109.22 0)
+			(effects
+				(font
+					(size 1.27 1.27)
+				)
+				(justify right)
 			)
 		)
 		(pin "CANL" input
-			(at 157.48 119.38 270)
-			(effects
-				(font
-					(size 1.27 1.27)
-				)
-				(justify left)
+			(at 173.99 102.87 0)
+			(effects
+				(font
+					(size 1.27 1.27)
+				)
+				(justify right)
 			)
 		)
@@
 		)
 		(pin "PRIMARY_HALL" input
-			(at 147.32 43.18 90)
+			(at 172.72 57.15 0)
 			(effects
 				(font
@@
 		)
 		(pin "SECONDARY_HALL" input
-			(at 157.48 43.18 90)
+			(at 172.72 60.96 0)
 			(effects
 				(font
@@
 		)
 		(pin "LIMIT" input
-			(at 138.43 43.18 90)
+			(at 172.72 53.34 0)
 			(effects
 				(font
@@
 		(pin "MISO" input
 			(at 161.29 72.39 270)
+			(effects
+				(font
+					(size 1.27 1.27)
+				)
+				(justify left)
+			)
+		)
+		(pin "S" input
+			(at 139.7 72.39 270)
 			(effects
 				(font
@@
 	)
 	(sheet
-		(at 194.31 46.99)
+		(at 228.6 95.25)
 		(size 45.72 17.78)
 		(exclude_from_sim no)
@@
 		)
 		(property "Sheetname" "Power"
-			(at 194.31 46.2784 0)
+			(at 228.6 94.5384 0)
 			(show_name no)
 			(do_not_autoplace no)
@@
 		)
 		(property "Sheetfile" "Power.kicad_sch"
-			(at 194.31 65.3546 0)
+			(at 228.6 113.6146 0)
 			(show_name no)
 			(do_not_autoplace no)
@@
 		)
 		(pin "12V_Motor_Driver" input
-			(at 194.31 55.88 180)
-			(effects
-				(font
+			(at 228.6 104.14 180)
+			(effects
+				(font

Commit message: initial placement
Other:
- sheet CAN ports: added none; removed S
- sheet MCU ports: added none; removed S
Changed lines of the file:
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@@
-			)
-		)
-		(pin "S" input
-			(at 139.7 92.71 90)
-			(effects
-				(font
-					(size 1.27 1.27)
-				)
-				(justify right)
 			)
 		)
@@
 			(effects
 				(font
-					(size 1.27 1.27)
-				)
-				(justify left)
-			)
-		)
-		(pin "S" input
-			(at 139.7 72.39 270)
-			(effects
-				(font

Commit message: Basic ERC fixed
Other:
- sheet CAN ports: added S; removed none
- sheet Connectors ports: added Sig1, Sig2; removed 12V_Motor_Driver
- sheet MCU ports: added Limit, Primary, S, Secondary, Sig1, Sig2; removed LIMIT, PRIMARY_HALL, SECONDARY_HALL
- sheet Power ports: added none; removed 12V_Motor_Driver
Changed lines of the file:
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@@
-	(wire
-		(pts
-			(xy 220.98 104.14) (xy 228.6 104.14)
-		)
-		(stroke
-			(width 0)
-			(type default)
-		)
-	)
 	(wire
 		(pts
@@
 	(wire
 		(pts
+			(xy 214.63 91.44) (xy 214.63 45.72)
+		)
+		(stroke
+			(width 0)
+			(type default)
+		)
+	)
+	(wire
+		(pts
+			(xy 214.63 45.72) (xy 172.72 45.72)
+		)
+		(stroke
+			(width 0)
+			(type default)
+		)
+	)
+	(wire
+		(pts
 			(xy 147.32 72.39) (xy 147.32 92.71)
 		)
@@
 	(wire
 		(pts
+			(xy 208.28 49.53) (xy 208.28 91.44)
+		)
+		(stroke
+			(width 0)
+			(type default)
+		)
+	)
+	(wire
+		(pts
+			(xy 142.24 72.39) (xy 142.24 92.71)
+		)
+		(stroke
+			(width 0)
+			(type default)
+		)
+	)
+	(wire
+		(pts
 			(xy 161.29 72.39) (xy 161.29 92.71)
 		)
@@
 		(pts
 			(xy 153.67 72.39) (xy 153.67 92.71)
+		)
+		(stroke
+			(width 0)
+			(type default)
+		)
+	)
+	(wire
+		(pts
+			(xy 172.72 49.53) (xy 208.28 49.53)
 		)
 		(stroke
@@
 			)
 		)
-		(pin "12V_Motor_Driver" input
-			(at 220.98 104.14 0)
-			(effects
-				(font
-					(size 1.27 1.27)
-				)
-				(justify right)
-			)
-		)
 		(pin "CANL" input
 			(at 181.61 102.87 180)
@@
 		(pin "Secondary" input
 			(at 193.04 91.44 90)
+			(effects
+				(font
+					(size 1.27 1.27)
+				)
+				(justify right)
+			)
+		)
+		(pin "Sig1" input
+			(at 214.63 91.44 90)
+			(effects
+				(font
+					(size 1.27 1.27)
+				)
+				(justify right)
+			)
+		)
+		(pin "Sig2" input
+			(at 208.28 91.44 90)
 			(effects
 				(font
@@
 			)
 		)
+		(pin "S" input
+			(at 142.24 92.71 90)
+			(effects
+				(font
+					(size 1.27 1.27)
+				)
+				(justify right)
+			)
+		)
 		(instances
 			(project "ecvt-controller"
@@
 			)
 		)
-		(pin "PRIMARY_HALL" input
-			(at 172.72 57.15 0)
-			(effects
-				(font
-					(size 1.27 1.27)
-				)
-				(justify right)
-			)
-		)
-		(pin "SECONDARY_HALL" input
-			(at 172.72 60.96 0)
-			(effects
-				(font
-					(size 1.27 1.27)
-				)
-				(justify right)
-			)
-		)
-		(pin "LIMIT" input
-			(at 172.72 53.34 0)
-			(effects
-				(font
-					(size 1.27 1.27)
-				)
-				(justify right)
-			)
-		)
 		(pin "CS0" input
 			(at 153.67 72.39 270)
@@
 				)
 				(justify left)
+			)
+		)
+		(pin "S" input
+			(at 142.24 72.39 270)
+			(effects
+				(font
+					(size 1.27 1.27)
+				)
+				(justify left)
+			)
+		)
+		(pin "Sig1" input
+			(at 172.72 45.72 0)
+			(effects
+				(font
+					(size 1.27 1.27)
+				)
+				(justify right)
+			)
+		)
+		(pin "Sig2" input
+			(at 172.72 49.53 0)
+			(effects
+				(font
+					(size 1.27 1.27)
+				)
+				(justify right)
+			)
+		)
+		(pin "Primary" input
+			(at 172.72 57.15 0)
+			(effects
+				(font
+					(size 1.27 1.27)
+				)
+				(justify right)
+			)
+		)
+		(pin "Secondary" input
+			(at 172.72 60.96 0)
+			(effects
+				(font
+					(size 1.27 1.27)
+				)
+				(justify right)
+			)
+		)
+		(pin "Limit" input
+			(at 172.72 53.34 0)
+			(effects
+				(font
+					(size 1.27 1.27)
+				)
+				(justify right)
 			)
 		)
@@
 	)
 	(sheet
-		(at 228.6 95.25)
+		(at 228.6 60.96)
 		(size 45.72 17.78)
 		(exclude_from_sim no)
@@
 		)
 		(property "Sheetname" "Power"
-			(at 228.6 94.5384 0)
+			(at 228.6 60.2484 0)
 			(show_name no)
 			(do_not_autoplace no)
@@
 		)
 		(property "Sheetfile" "Power.kicad_sch"
-			(at 228.6 113.6146 0)
+			(at 228.6 79.3246 0)
 			(show_name no)
 			(do_not_autoplace no)
@@
 			)
 		)
-		(pin "12V_Motor_Driver" input
-			(at 228.6 104.14 180)
-			(effects
-				(font
-					(size 1.27 1.27)
-				)
-				(justify left)
-			)
-		)

Commit message: ADC done
Other:
- added sheet ADC (ADC.kicad_sch)
- sheet Connectors ports: added AIN0, AIN1; removed none
- sheet MCU ports: added SCL, SDA; removed none

Commit message: Capacitors !!!!
Changed lines of the file:
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@@
 	)
 	(sheet
-		(at 125.73 139.7)
+		(at 74.93 69.85)
 		(size 45.72 17.78)
 		(exclude_from_sim no)
@@
 		)
 		(property "Sheetname" "Power"
-			(at 125.73 138.9884 0)
+			(at 74.93 69.1384 0)
 			(show_name no)
 			(do_not_autoplace no)
@@
 		)
 		(property "Sheetfile" "Power.kicad_sch"
-			(at 125.73 158.0646 0)
+			(at 74.93 88.2146 0)
 			(show_name no)
 			(do_not_autoplace no)

Commit message: Done  danadan done done da da
Other:
- sheet CAN ports: added none; removed S
- sheet MCU ports: added none; removed S
Changed lines of the file:
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@@
-	(wire
-		(pts
-			(xy 135.89 72.39) (xy 135.89 92.71)
-		)
-		(stroke
-			(width 0)
-			(type default)
-		)
-	)
 	(wire
 		(pts
@@
 			)
 		)
-		(pin "S" input
-			(at 135.89 92.71 90)
-			(effects
-				(font
-					(size 1.27 1.27)
-				)
-				(justify right)
-			)
-		)
 		(instances
 			(project "ecvt-controller"
@@
 			(effects
 				(font
-					(size 1.27 1.27)
-				)
-				(justify left)
-			)
-		)
-		(pin "S" input
-			(at 135.89 72.39 270)
-			(effects
-				(font
