File: boards/ecvt-controller/ecvt-controller/ecvt-controller.kicad_pcb (KiCad board)
At the start: 2 copper layers, 121.5 x 65 mm, 40 parts, among them J1 Conn_02x20_Odd_Even, J3 1720420206, J4 1720420206, J5 917786-1, J6 917780-1, Q1 Q_PMOS, SW1 SW_SPST, SW2 SW_SPST, U1 TJA1051T-3, U2 TSR3-2450N, U3 MCP2515-xSO, U5 ACT45B-101-2P-TL003, U6 PESD2CAN,215, Y1 Crystal

Commit message: Pre-DR
Parts:
- removed J3: 1720420206, Molex_SuperSabre:CONN_SD-172042-001_02_BL_MOL
- J1: moved to B.Cu
- J4: value 1720420206 -> 15311026; footprint Molex_SuperSabre:CONN_SD-172042-001_02_BL_MOL -> baja_footprint_library:MOLEX_15311026
- moved C20 115.4 mm to (71.0, 83.0), turned to 180 degrees
- moved C19 115.3 mm to (71.0, 81.0), turned to 180 degrees
- moved D6 99.2 mm to (106.5, 73.8), turned to 90 degrees
- moved D7 99.2 mm to (106.5, 76.3), turned to 90 degrees
- moved D8 99.1 mm to (106.5, 79.0), turned to 90 degrees
- moved C14 96.4 mm to (106.5, 60.5), turned to 90 degrees
- moved C12 86.2 mm to (115.5, 60.5), turned to 90 degrees
- moved C13 84.2 mm to (118.5, 60.5), turned to 90 degrees
- moved J5 72.7 mm to (91.0, 63.8)
- moved R3 72.5 mm to (127.0, 85.0), turned to -90 degrees
- moved J4 45.4 mm to (124.2, 106.6)
- moved J6 25.3 mm to (55.6, 81.8), turned to -90 degrees
- moved SW2 21.1 mm to (63.2, 76.0)
- moved Q1 19.2 mm to (121.8, 88.5)
- moved SW1 18.8 mm to (70.8, 87.5), turned to 180 degrees
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Connections:
- D6 pad 1: /MCU/GPIO23 -> /MCU/GPIO17
- D7 pad 1: /MCU/GPIO24 -> /MCU/GPIO27
- D8 pad 1: /MCU/GPIO25 -> /MCU/GPIO22
- F1 pad 1: /Connectors/12V_Motor_Driver -> Net-(F1-Pad1)
- J4 pad 1: /Connectors/12V_Motor_Driver -> +12V
- J5 pad 2: /MCU/GPIO23 -> /MCU/GPIO17
- J5 pad 5: /MCU/GPIO24 -> /MCU/GPIO27
- J5 pad 8: /MCU/GPIO25 -> /MCU/GPIO22
Routing:
- net /CAN/CANL: track 0.00 -> 25.9 mm
- net /CAN/CANH: track 0.00 -> 22.2 mm
- net +5V: track 0.00 -> 16.6 mm
- net Net-(U1-RXD): track 0.00 -> 12.8 mm
- net /MCU/GPIO5: track 0.00 -> 11.7 mm
- net Net-(U2-Vin): track 0.00 -> 10.3 mm
- net Net-(U1-CANH): track 0.00 -> 9.45 mm
- net +3.3V: track 0.00 -> 8.02 mm
- net /MCU/GPIO10: track 0.00 -> 7.99 mm
- net Net-(U1-CANL): track 0.00 -> 7.82 mm
- net /MCU/GPIO11: track 0.00 -> 7.21 mm
- net Net-(SW2-A): track 0.00 -> 5.43 mm
- net Net-(SW1-B): track 0.00 -> 5.41 mm
- net Net-(C21-Pad2): track 0.00 -> 5.10 mm
- net Net-(U3-OSC2): track 0.00 -> 4.74 mm
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Other:
- board size 121.5 x 65 mm -> 90 x 65 mm

Commit message: removed old version
Parts:
- moved D8 25.8 mm to (82.5, 69.5)
- moved D7 17.9 mm to (90.0, 69.5)
- moved D6 10.2 mm to (97.5, 69.2)
- moved J4 0.71 mm to (123.7, 106.1)
- moved Q1 0.54 mm to (121.3, 88.8)
Connections:
- net Net-(F1-Pad1) renamed /Power/S
- net Net-(Q1-PadG) renamed /Power/G
- C22 pad 1: Net-(U2-Vin) -> GND
- C22 pad 2: GND -> Net-(U2-Vin)
Routing:
- net Net-(U1-RXD): track 12.8 -> 0.00 mm
- net Net-(U1-CANH): track 9.45 -> 7.82 mm

Commit message: Rough Placement
no traces, slightly worries about 5V and 3.3V
Parts:
- removed C18, C21, C22, C23: 0.1 µF, Capacitor_SMD:C_0603_1608Metric_Pad1.08x0.95mm_HandSolder
- removed C19, C20: 220 pF, Capacitor_SMD:C_0603_1608Metric_Pad1.08x0.95mm_HandSolder
- removed Y1: Crystal, Crystal:Crystal_SMD_5032-2Pin_5.0x3.2mm_HandSoldering
- added C1: 30pF, Capacitor_SMD:C_0603_1608Metric_Pad1.08x0.95mm_HandSolder, F.Cu at (88.5, 88.0)
- added C2: 30pF, Capacitor_SMD:C_0603_1608Metric_Pad1.08x0.95mm_HandSolder, F.Cu at (88.5, 91.5)
- added C3: 4.7µF, Capacitor_SMD:C_0805_2012Metric_Pad1.18x1.45mm_HandSolder, F.Cu at (115.5, 60.0)
- added C4: 0.1 µF, Capacitor_SMD:C_0603_1608Metric_Pad1.08x0.95mm_HandSolder, F.Cu at (106.5, 60.5)
- added C5: 0.1 µF, Capacitor_SMD:C_0603_1608Metric_Pad1.08x0.95mm_HandSolder, F.Cu at (118.0, 60.0)
- added C6: 0.1 µF, Capacitor_SMD:C_0603_1608Metric_Pad1.08x0.95mm_HandSolder, F.Cu at (118.5, 82.5)
- added C7: 0.1 µF, Capacitor_SMD:C_0603_1608Metric_Pad1.08x0.95mm_HandSolder, F.Cu at (115.0, 72.0)
- added C8: 0.1 µF, Capacitor_SMD:C_0603_1608Metric_Pad1.08x0.95mm_HandSolder, F.Cu at (143.7, 93.4)
- added C9: 0.1 µF, Capacitor_SMD:C_0603_1608Metric_Pad1.08x0.95mm_HandSolder, F.Cu at (143.7, 95.9)
- added D1: 1N4148, Diode_THT:D_DO-35_SOD27_P7.62mm_Horizontal, F.Cu at (150.6, 99.0)
- added D2: D_TVS, Diode_SMD:D_SOD-323_HandSoldering, F.Cu at (83.5, 64.5)
- added D3: D_TVS, Diode_SMD:D_SOD-323_HandSoldering, F.Cu at (75.5, 64.5)
- added D4: D_TVS, Diode_SMD:D_SOD-323_HandSoldering, F.Cu at (68.0, 64.5)
- added D5: D_TVS, Diode_SMD:D_SOD-323_HandSoldering, F.Cu at (99.5, 101.0)
- added D9: D_Zener, Diode_THT:D_P600_R-6_P12.70mm_Horizontal, F.Cu at (130.0, 98.3)
- added J2: 917782-1, baja-common-parts:CON4_1X4_P100, F.Cu at (101.0, 58.4)
- added J3: 917782-1, baja-common-parts:CON4_1X4_P100, F.Cu at (100.8, 105.9)
- added PS1: TSR_3-2450N, baja-common-parts:CONV_TSR_3-2450N, F.Cu at (120.0, 74.0)
- added R1: 10k, Resistor_SMD:R_0603_1608Metric_Pad0.98x0.95mm_HandSolder, F.Cu at (93.2, 66.5)
- added R10: 10k, Resistor_SMD:R_0603_1608Metric_Pad0.98x0.95mm_HandSolder, F.Cu at (152.4, 95.9)
- added R2: 15k, Resistor_SMD:R_0603_1608Metric_Pad0.98x0.95mm_HandSolder, F.Cu at (93.2, 68.5)
- added R8: 10k, Resistor_SMD:R_0603_1608Metric_Pad0.98x0.95mm_HandSolder, F.Cu at (97.8, 66.5)
- added R9: 15k, Resistor_SMD:R_0603_1608Metric_Pad0.98x0.95mm_HandSolder, F.Cu at (97.8, 68.5)
- added Y2: ABM3-16.000MHZ-D2Y-T, baja_footprint_library:XTAL_ABM3-16.000MHZ-D2Y-T, F.Cu at (91.5, 89.5)
- C10, C11: value 22pF -> 0.1 µF; footprint Capacitor_SMD:C_0805_2012Metric_Pad1.18x1.45mm_HandSolder -> Capacitor_SMD:C_0603_1608Metric_Pad1.08x0.95mm_HandSolder
- C12, C15: footprint Capacitor_SMD:C_0603_1608Metric_Pad1.08x0.95mm_HandSolder -> Capacitor_SMD:C_0805_2012Metric_Pad1.18x1.45mm_HandSolder
- C16: value 0.1 µF -> 220pF
- C17: value 4.7µF -> 220pF
- D6, D7, D8: value DF2S5M4CTL3FCT-ND -> D_TVS; footprint Diode_SMD:D_SOD-882 -> Diode_SMD:D_SOD-323_HandSoldering
- F1: footprint Fuse:Fuse_1206_3216Metric -> Fuse:Fuse_1206_3216Metric_Pad1.42x1.75mm_HandSolder
- Q1: value Q_PMOS -> Q_PMOS_GDS
- R3: footprint Resistor_SMD:R_0603_1608Metric_Pad0.98x0.95mm_HandSolder -> Resistor_SMD:R_0805_2012Metric_Pad1.20x1.40mm_HandSolder
- R4: value 10k -> 1k; footprint Resistor_SMD:R_0603_1608Metric_Pad0.98x0.95mm_HandSolder -> Resistor_SMD:R_0805_2012Metric_Pad1.20x1.40mm_HandSolder
- R5, R6: footprint Resistor_SMD:R_1206_3216Metric_Pad1.30x1.75mm_HandSolder -> Resistor_SMD:R_0603_1608Metric_Pad0.98x0.95mm_HandSolder
- U2: value TSR3-2450N -> ADS1115IDGS; footprint Converter_DCDC:Converter_DCDC_TRACO_TSR2-24xxN_TSR2-24xxxN_THT -> Package_SO:TSSOP-10_3x3mm_P0.5mm
- U6: footprint Package_TO_SOT_SMD:SOT-23 -> Package_TO_SOT_SMD:SOT-23-3
- moved R6 90.8 mm to (152.4, 93.4)
- moved R5 90.2 mm to (152.4, 90.9), turned to 0 degrees
- moved C15 76.2 mm to (157.0, 91.7), turned to 0 degrees
- moved C16 70.3 mm to (148.0, 95.9), turned to 0 degrees
- moved C17 64.2 mm to (152.4, 88.4)
- moved C11 62.5 mm to (148.0, 90.9), turned to 0 degrees
- moved C10 62.5 mm to (148.0, 88.4), turned to 0 degrees
- moved C14 53.0 mm to (148.0, 93.4), turned to 0 degrees
- moved R4 52.4 mm to (156.9, 94.6), turned to 0 degrees
- moved C12 50.1 mm to (157.0, 88.7), turned to 0 degrees
- moved D6 32.0 mm to (94.5, 101.0), turned to 0 degrees
- moved C13 21.3 mm to (100.2, 71.5), turned to 180 degrees
- moved U2 19.3 mm to (101.8, 67.5), turned to -90 degrees
- moved J5 13.8 mm to (78.0, 59.0)
- moved D8 11.9 mm to (93.2, 64.5), turned to 0 degrees
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Connections:
- net /MCU/GPIO10 renamed /CAN/SI
- net /MCU/GPIO11 renamed /CAN/SCK
- net /MCU/GPIO5 renamed /CAN/INT
- net /MCU/GPIO8 renamed /CAN/CS
- net /MCU/GPIO9 renamed /CAN/SO
- C10 pad 1: GND -> +3.3V
- C10 pad 2: Net-(U3-OSC2) -> GND
- C11 pad 1: GND -> +5V
- C11 pad 2: Net-(U3-OSC1) -> GND
- C13 pad 1: +5V -> +3.3V
- C14 pad 1: +3.3V -> Net-(C14-Pad1)
- C16 pad 1: +3.3V -> /CAN/CANH
- C17 pad 1: +5V -> /CAN/CANL
- D6 pad 1: /MCU/GPIO17 -> GND
- D6 pad 2: GND -> /Connectors/Sig2
- D7 pad 1: /MCU/GPIO27 -> GND
- D7 pad 2: GND -> /ADC/AIN1
- D8 pad 1: /MCU/GPIO22 -> GND
- D8 pad 2: GND -> /ADC/AIN0
- F1 pad 1: /Power/S -> Net-(Q1-S)
- F1 pad 2: Net-(U2-Vin) -> Net-(PS1-+VIN)
- J1 pad 10: /MCU/GPIO15 -> unconnected-(J1-Pin_10-Pad10)
- J1 pad 11: /MCU/GPIO17 -> /Connectors/Primary
- J1 pad 12: /MCU/GPIO18 -> unconnected-(J1-Pin_12-Pad12)
- J1 pad 13: /MCU/GPIO27 -> /Connectors/Secondary
- J1 pad 15: /MCU/GPIO22 -> /Connectors/Limit
- J1 pad 16: /MCU/GPIO23 -> unconnected-(J1-Pin_16-Pad16)
- J1 pad 18: /MCU/GPIO24 -> unconnected-(J1-Pin_18-Pad18)
- J1 pad 22: /MCU/GPIO25 -> unconnected-(J1-Pin_22-Pad22)
- J1 pad 26: /MCU/GPIO7 -> unconnected-(J1-Pin_26-Pad26)
- J1 pad 27: /MCU/GPIO0 -> unconnected-(J1-Pin_27-Pad27)
- J1 pad 28: /MCU/GPIO1 -> unconnected-(J1-Pin_28-Pad28)
- J1 pad 3: /MCU/GPIO2 -> /ADC/SDA
- J1 pad 31: /MCU/GPIO6 -> /CAN/S
- J1 pad 32: /MCU/GPIO12 -> unconnected-(J1-Pin_32-Pad32)
- J1 pad 33: /MCU/GPIO13 -> unconnected-(J1-Pin_33-Pad33)
- J1 pad 35: /MCU/GPIO19 -> /Connectors/Sig1
- J1 pad 36: /MCU/GPIO16 -> unconnected-(J1-Pin_36-Pad36)
- J1 pad 37: /MCU/GPIO26 -> /Connectors/Sig2
- J1 pad 38: /MCU/GPIO20 -> unconnected-(J1-Pin_38-Pad38)
- J1 pad 40: /MCU/GPIO21 -> unconnected-(J1-Pin_40-Pad40)
- J1 pad 5: /MCU/GPIO3 -> /ADC/SCL
- J1 pad 7: /MCU/GPIO4 -> unconnected-(J1-Pin_7-Pad7)
- J1 pad 8: /MCU/GPIO14 -> unconnected-(J1-Pin_8-Pad8)
- J5 pad 2: /MCU/GPIO17 -> /Connectors/Primary
- J5 pad 5: /MCU/GPIO27 -> /Connectors/Secondary
- J5 pad 8: /MCU/GPIO22 -> /Connectors/Limit
- Q1 pad 1: (no net) -> Net-(Q1-G)
- Q1 pad 2: (no net) -> +12V
- Q1 pad 3: (no net) -> Net-(Q1-S)
- R3 pad 1: /Power/G -> Net-(Q1-G)
- R4 pad 1: +3.3V -> /CAN/RESET
- R4 pad 2: Net-(U3-~{RESET}) -> Net-(D1-A)
- R5 pad 1: Net-(C21-Pad2) -> Net-(SW1-B)
- R5 pad 2: Net-(SW1-B) -> Net-(C14-Pad1)
- R6 pad 1: Net-(SW2-A) -> Net-(C14-Pad1)
- R6 pad 2: Net-(C21-Pad2) -> Net-(SW2-A)
- U1 pad 8: GND -> /CAN/S
- U2 pad 1: Net-(U2-Vin) -> GND
- U2 pad 2: GND -> unconnected-(U2-ALERT/RDY-Pad2)
- U2 pad 3: +5V -> GND
- U3 pad 17: Net-(U3-~{RESET}) -> /CAN/RESET
Routing:
- net /CAN/CANL: track 25.9 -> 0.00 mm
- net /CAN/CANH: track 22.2 -> 0.00 mm
- net +5V: track 16.6 -> 0.00 mm
- net /CAN/INT: track 11.7 -> 0.00 mm
- net Net-(U2-Vin): track 10.3 -> 0.00 mm
- net +3.3V: track 8.02 -> 0.00 mm
- net /CAN/SI: track 7.99 -> 0.00 mm
- net Net-(U1-CANL): track 7.82 -> 0.00 mm
- net Net-(U1-CANH): track 7.82 -> 0.00 mm
- net /CAN/SCK: track 7.21 -> 0.00 mm
- net Net-(SW2-A): track 5.43 -> 0.00 mm
- net Net-(SW1-B): track 5.41 -> 0.00 mm
- net Net-(C21-Pad2): track 5.10 -> 0.00 mm
- net Net-(U3-OSC2): track 4.74 -> 0.00 mm
- net Net-(U1-TXD): track 4.70 -> 0.00 mm
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
Commit message: layout planned !
Parts:
- moved C17 81.7 mm to (72.5, 105.5), turned to 180 degrees
- moved R6 79.2 mm to (73.5, 101.0), turned to -90 degrees
- moved R5 76.0 mm to (77.0, 101.0), turned to 90 degrees
- moved C12 75.0 mm to (83.0, 76.0), turned to 180 degrees
- moved C14 73.0 mm to (75.1, 98.0)
- moved C15 70.8 mm to (87.5, 78.0)
- moved C16 70.7 mm to (78.0, 106.0)
- moved C11 66.3 mm to (83.0, 78.0), turned to 180 degrees
- moved D1 63.5 mm to (87.2, 95.5)
- moved C10 62.3 mm to (87.0, 76.0)
- moved R4 58.9 mm to (98.0, 94.5), turned to 180 degrees
- moved R10 54.4 mm to (98.0, 96.5), turned to 180 degrees
- moved C9 49.2 mm to (94.5, 98.0), turned to 180 degrees
- moved C8 39.2 mm to (106.5, 80.9), turned to 90 degrees
- moved J6 34.7 mm to (75.3, 110.4), turned to 0 degrees
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Connections:
- D5 pad 2: /Connectors/Sig1 -> /Connectors/Sig2
- D6 pad 2: /Connectors/Sig2 -> /Connectors/Sig1
- J3 pad 2: /Connectors/Sig1 -> /Connectors/Sig2
- J3 pad 3: /Connectors/Sig2 -> /Connectors/Sig1
Routing:
- net +3.3V: track 0.00 -> 145.2 mm, vias 0 -> 2
- net +5V: track 0.00 -> 107.9 mm
- net /Connectors/Limit: track 0.00 -> 52.5 mm
- net /Connectors/Secondary: track 0.00 -> 44.0 mm
- net /Connectors/Primary: track 0.00 -> 36.2 mm
- net /CAN/CANL: track 0.00 -> 27.0 mm
- net /CAN/CANH: track 0.00 -> 26.8 mm
- net /ADC/AIN0: track 0.00 -> 21.5 mm
- net +12V: track 0.00 -> 20.8 mm
- net /Connectors/Sig1: track 0.00 -> 17.2 mm
- net /Connectors/Sig2: track 0.00 -> 15.4 mm
- net Net-(U1-CANL): track 0.00 -> 15.1 mm
- net /ADC/AIN1: track 0.00 -> 14.9 mm
- net Net-(U1-CANH): track 0.00 -> 14.8 mm
- net /CAN/CS: track 0.00 -> 13.8 mm
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Other:
- board size 90 x 65 mm -> 79.5 x 65 mm

Commit message: Done  danadan done done da da
Parts:
- moved C5 1.00 mm to (117.0, 60.0)
- moved C3 0.50 mm to (115.0, 60.0)
- moved PS1 0.50 mm to (120.0, 73.5)
Connections:
- C8 pad 1: +3.3V -> +3.3V(v2)
- J1 pad 17: +3.3V -> +3.3V(v2)
- J1 pad 31: /CAN/S -> unconnected-(J1-Pin_31-Pad31)
- R1 pad 2: /ADC/AIN0 -> /ADC/AIN0_in
- R2 pad 1: /ADC/AIN0 -> /ADC/AIN0_in
- R8 pad 2: /ADC/AIN1 -> /ADC/AIN1_in
- R9 pad 1: /ADC/AIN1 -> /ADC/AIN1_in
- U1 pad 8: /CAN/S -> GND
- U2 pad 4: /ADC/AIN0 -> /ADC/AIN0_in
- U2 pad 5: /ADC/AIN1 -> /ADC/AIN1_in
- U3 pad 18: +3.3V -> +3.3V(v2)
Routing:
- net GND: track 0.00 -> 70.0 mm, vias 0 -> 46
- net +3.3V: track 145.2 -> 158.8 mm
- net /ADC/AIN0_in: track 0.00 -> 12.6 mm
- net /ADC/AIN0: track 21.5 -> 10.2 mm
- net /ADC/SDA: track 0.00 -> 10.1 mm
- net +3.3V(v2): track 0.00 -> 8.43 mm
- net /ADC/SCL: track 0.00 -> 8.06 mm
- net Net-(U3-OSC2): track 0.00 -> 7.35 mm
- net Net-(U3-OSC1): track 0.00 -> 6.99 mm
- net /ADC/AIN1_in: track 0.00 -> 6.98 mm
- net +5V: track 107.9 -> 113.9 mm
- net /ADC/AIN1: track 14.9 -> 9.29 mm
- net /Connectors/Sig2: track 15.4 -> 20.3 mm
- net /Connectors/Sig1: track 17.2 -> 22.1 mm
- net +12V: track 20.8 -> 21.6 mm
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- added copper zone on B.Cu, net GND
Other:
- outline, holes or cut-outs redrawn

Commit message: with logo
Parts:
- added G***: LOGO, baja_footprint_library:baja_logo_footprint, F.Cu at (66.2, 76.0)
Other:
- board text added: "ECVT Controller v1 MANASH DUGAR ALEX HALLEY"
